File: attenuverters/attenuverters.kicad_pcb (KiCad board)
At the start: 2 copper layers, 42 parts, among them J1 C1, J2 C2, U1 OPA4991, U2 TL072

Commit message: Attvert board layout
Parts:
- added J3: C5, Connector_PinSocket_2.54mm:PinSocket_1x03_P2.54mm_Vertical, F.Cu at (73.7, 76.2)
- added J4: C2, Connector_PinSocket_2.54mm:PinSocket_1x03_P2.54mm_Vertical, F.Cu at (73.7, 48.3)
- added J5: C4, Connector_PinSocket_2.54mm:PinSocket_1x03_P2.54mm_Vertical, F.Cu at (73.7, 63.5)
- added J6: C6, Connector_PinSocket_2.54mm:PinSocket_1x03_P2.54mm_Vertical, F.Cu at (38.1, 76.2)
- added kibuzzard-65FD5706: G***, kibuzzard-65FD5706, F.Cu at (66.0, 88.8)
- added kibuzzard-65FD5706: G***, kibuzzard-65FD5706, F.Cu at (66.0, 40.8)
- added kibuzzard-65FD570C: G***, kibuzzard-65FD570C, F.Cu at (48.3, 40.1)
- added kibuzzard-65FD570C: G***, kibuzzard-65FD570C, F.Cu at (48.1, 89.4)
- J1: footprint Connector_PinSocket_2.54mm:PinSocket_1x10_P2.54mm_Vertical -> Connector_PinSocket_2.54mm:PinSocket_1x03_P2.54mm_Vertical
- J2: value C2 -> C3; footprint Connector_PinSocket_2.54mm:PinSocket_1x10_P2.54mm_Vertical -> Connector_PinSocket_2.54mm:PinSocket_1x03_P2.54mm_Vertical
- moved J2 37.0 mm to (38.1, 63.5)
- moved R16 5.84 mm to (60.2, 70.7)
- moved J1 5.08 mm to (38.1, 48.3)
- moved R20 3.91 mm to (60.2, 66.8)
- turned R10 to 90 degrees
Connections:
- J1 pad 1: /+9V -> /In1
- J1 pad 3: /+4.5V -> /Out1
- RV3 pad 0: Net-(R6-Pad1) -> /GND
- RV4 pad 0: Net-(R8-Pad1) -> /GND
Routing:
- net /In1: track 0.00 -> 67.0 mm
- net /Out2: track 0.00 -> 59.8 mm, vias 0 -> 1
- net /Out1: track 0.00 -> 48.5 mm, vias 0 -> 1
- net /+9V: track 0.00 -> 46.0 mm, vias 0 -> 3
- net /In2: track 0.00 -> 43.6 mm, vias 0 -> 1
- net Net-(D1-Pad1): track 0.00 -> 38.4 mm
- net Net-(D1-Pad2): track 0.00 -> 37.1 mm
- net Net-(D2-Pad1): track 0.00 -> 36.0 mm
- net Net-(D2-Pad2): track 0.00 -> 35.6 mm
- net Net-(C3-Pad1): track 0.00 -> 28.4 mm
- net Net-(C3-Pad2): track 0.00 -> 28.1 mm
- net Net-(RV2-Pad2): track 0.00 -> 24.2 mm
- net Net-(RV1-Pad2): track 0.00 -> 21.3 mm
- net Net-(C4-Pad1): track 0.00 -> 18.7 mm
- net Net-(C2-Pad1): track 0.00 -> 14.7 mm
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- added copper zone on B.Cu, net /+4.5V
- added copper zone on F.Cu, net /+9V
- added copper zone on In1.Cu, net /GND
- added copper zone on In2.Cu, net /GND
Other:
- board outline added: 40.6 x 58.4 mm
- copper layers 2 -> 4

Commit message: Attvert graphics
Parts:
- added G***: LOGO, LOGO, B.Cu at (55.9, 84.5)
- added REF**: OSHW-Logo2_7.3x6mm_SilkScreen, Symbol:OSHW-Logo2_7.3x6mm_SilkScreen, B.Cu at (55.9, 44.5)
- added kibuzzard-65FDA4E4: G***, kibuzzard-65FDA4E4, B.Cu at (44.5, 48.3)
- added kibuzzard-65FDA4EE: G***, kibuzzard-65FDA4EE, B.Cu at (44.5, 50.8)
- added kibuzzard-65FDA500: G***, kibuzzard-65FDA500, B.Cu at (41.3, 63.5)
- added kibuzzard-65FDA507: G***, kibuzzard-65FDA507, B.Cu at (41.3, 66.0)
- added kibuzzard-65FDA513: G***, kibuzzard-65FDA513, B.Cu at (41.3, 68.6)
- added kibuzzard-65FDA527: G***, kibuzzard-65FDA527, B.Cu at (44.5, 76.2)
- added kibuzzard-65FDA52F: G***, kibuzzard-65FDA52F, B.Cu at (44.5, 78.7)
- added kibuzzard-65FDA541: G***, kibuzzard-65FDA541, B.Cu at (44.5, 81.3)
- added kibuzzard-65FDA56F: G***, kibuzzard-65FDA56F, B.Cu at (44.5, 53.3)
- added kibuzzard-65FDA57B: G***, kibuzzard-65FDA57B, B.Cu at (70.5, 48.3)
- added kibuzzard-65FDA584: G***, kibuzzard-65FDA584, B.Cu at (70.5, 50.8)
- added kibuzzard-65FDA598: G***, kibuzzard-65FDA598, B.Cu at (70.5, 63.5)
- added kibuzzard-65FDA5A0: G***, kibuzzard-65FDA5A0, B.Cu at (70.5, 66.0)
- added kibuzzard-65FDA5A8: G***, kibuzzard-65FDA5A8, B.Cu at (70.5, 68.6)
- added kibuzzard-65FDA5B3: G***, kibuzzard-65FDA5B3, B.Cu at (70.5, 76.2)
- added kibuzzard-65FDA5BA: G***, kibuzzard-65FDA5BA, B.Cu at (70.5, 78.7)
- added kibuzzard-65FDA5C9: G***, kibuzzard-65FDA5C9, B.Cu at (70.5, 81.3)
- added kibuzzard-65FDA5D6: G***, kibuzzard-65FDA5D6, B.Cu at (70.5, 53.3)
Other:
- board text added: "1"
- board text added: "2"
- board text added: "3"
- board text added: "4"
- board text added: "5"
- board text added: "6"
- board text added: "7"
- board text added: "8"
- board text added: "9"
- board text added: "pedalmarkt.com"

Commit message: AttVert pre-jlc
Other:
- board text added: "JLCJLCJLCJLC"

Commit message: AttVert JLCPCB order
Routing:
- net Net-(C1-Pad1): track 14.0 -> 18.0 mm
