File: attenuverters/attenuverters.kicad_pcb (KiCad board)
At the start: 4 copper layers, 40.6 x 58.4 mm, 70 parts, among them J1 C1, J2 C3, J3 C5, J4 C2, J5 C4, J6 C6, U1 OPA4991, U2 TL072

Commit message: Attvert version on the board
Other:
- board text added: "v1rev1"
Changed lines of the file:
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@@
     (effects (font (size 0.8 0.8) (thickness 0.12)) (justify mirror))
+  )
+  (gr_text "v1rev1" (at 73.66 40.64 270) (layer "B.SilkS")
+    (effects (font (size 0.9 0.9) (thickness 0.15)) (justify mirror))
   )
   (gr_text "1" (at 75.184 48.26) (layer "F.SilkS")

Commit message: wip
Parts:
- removed kibuzzard-65FDA4E4: G***, kibuzzard-65FDA4E4
- removed kibuzzard-65FDA4EE: G***, kibuzzard-65FDA4EE
- removed kibuzzard-65FDA500: G***, kibuzzard-65FDA500
- removed kibuzzard-65FDA507: G***, kibuzzard-65FDA507
- removed kibuzzard-65FDA513: G***, kibuzzard-65FDA513
- removed kibuzzard-65FDA527: G***, kibuzzard-65FDA527
- removed kibuzzard-65FDA52F: G***, kibuzzard-65FDA52F
- removed kibuzzard-65FDA541: G***, kibuzzard-65FDA541
- removed kibuzzard-65FDA56F: G***, kibuzzard-65FDA56F
- removed kibuzzard-65FDA57B: G***, kibuzzard-65FDA57B
- removed kibuzzard-65FDA584: G***, kibuzzard-65FDA584
- removed kibuzzard-65FDA598: G***, kibuzzard-65FDA598
- removed kibuzzard-65FDA5A0: G***, kibuzzard-65FDA5A0
- removed kibuzzard-65FDA5A8: G***, kibuzzard-65FDA5A8
- removed kibuzzard-65FDA5B3: G***, kibuzzard-65FDA5B3
- removed kibuzzard-65FDA5BA: G***, kibuzzard-65FDA5BA
- removed kibuzzard-65FDA5C9: G***, kibuzzard-65FDA5C9
- removed kibuzzard-65FDA5D6: G***, kibuzzard-65FDA5D6
- added kibuzzard-672CA9D7: G***, kibuzzard-672CA9D7, B.Cu at (44.9, 48.8)
- added kibuzzard-672CA9E5: G***, kibuzzard-672CA9E5, B.Cu at (45.0, 50.8)
- added kibuzzard-672CA9F1: G***, kibuzzard-672CA9F1, B.Cu at (44.9, 52.9)
- added kibuzzard-672CAA17: G***, kibuzzard-672CAA17, B.Cu at (41.3, 66.0)
- added kibuzzard-672CAA1B: G***, kibuzzard-672CAA1B, B.Cu at (41.3, 63.5)
- added kibuzzard-672CAA21: G***, kibuzzard-672CAA21, B.Cu at (41.3, 68.6)
- added kibuzzard-672CAA28: G***, kibuzzard-672CAA28, B.Cu at (44.9, 76.5)
- added kibuzzard-672CAA2D: G***, kibuzzard-672CAA2D, B.Cu at (45.0, 78.8)
- added kibuzzard-672CAA31: G***, kibuzzard-672CAA31, B.Cu at (44.9, 80.9)
- added kibuzzard-672CAA40: G***, kibuzzard-672CAA40, B.Cu at (70.1, 80.9)
- added kibuzzard-672CAA46: G***, kibuzzard-672CAA46, B.Cu at (69.9, 78.7)
- added kibuzzard-672CAA4A: G***, kibuzzard-672CAA4A, B.Cu at (69.9, 76.5)
- added kibuzzard-672CAA50: G***, kibuzzard-672CAA50, B.Cu at (70.5, 68.6)
- added kibuzzard-672CAA54: G***, kibuzzard-672CAA54, B.Cu at (70.5, 66.0)
- added kibuzzard-672CAA58: G***, kibuzzard-672CAA58, B.Cu at (70.5, 63.5)
- added kibuzzard-672CAA5E: G***, kibuzzard-672CAA5E, B.Cu at (70.1, 52.9)
- added kibuzzard-672CAA64: G***, kibuzzard-672CAA64, B.Cu at (69.9, 50.8)
- added kibuzzard-672CAA68: G***, kibuzzard-672CAA68, B.Cu at (69.9, 48.8)
Other:
- board text added: "v1rev2"
- board text removed: "v1rev1"
