File: attenuverters/attenuverters.kicad_sch (KiCad schematic)
At the start: 42 parts, among them J1 C1, J2 C2, U1 OPA4991, U2 TL072

Commit message: Attvert board layout
Parts:
- removed J1: C1, Connector_PinSocket_2.54mm:PinSocket_1x10_P2.54mm_Vertical, symbol Connector:Conn_01x10_Male
- removed J2: C2, Connector_PinSocket_2.54mm:PinSocket_1x10_P2.54mm_Vertical, symbol Connector:Conn_01x10_Male
- added J1: C1, Connector_PinSocket_2.54mm:PinSocket_1x03_P2.54mm_Vertical, symbol Connector:Conn_01x03_Male
- added J2: C3, Connector_PinSocket_2.54mm:PinSocket_1x03_P2.54mm_Vertical, symbol Connector:Conn_01x03_Male
- added J3: C5, Connector_PinSocket_2.54mm:PinSocket_1x03_P2.54mm_Vertical, symbol Connector:Conn_01x03_Male
- added J4: C2, Connector_PinSocket_2.54mm:PinSocket_1x03_P2.54mm_Vertical, symbol Connector:Conn_01x03_Male
- added J5: C4, Connector_PinSocket_2.54mm:PinSocket_1x03_P2.54mm_Vertical, symbol Connector:Conn_01x03_Male
- added J6: C6, Connector_PinSocket_2.54mm:PinSocket_1x03_P2.54mm_Vertical, symbol Connector:Conn_01x03_Male
Connections:
- net +4.5V: now also J2.3 (Pin_3), J5.3 (Pin_3)
- net +9V: now also J2.1 (Pin_1), J5.1 (Pin_1)
- net GND: now also RV3.0 (ShieldPin), RV4.0 (ShieldPin), J1.2 (Pin_2), J2.2 (Pin_2), J3.2 (Pin_2), J4.2 (Pin_2), J5.2 (Pin_2), J6.2 (Pin_2)
- net In1: now also J1.1 (Pin_1), J4.1 (Pin_1)
- net In2: now also J3.1 (Pin_1), J6.1 (Pin_1)
- net Out1: now also J1.3 (Pin_3), J4.3 (Pin_3)
- net Out2: now also J3.3 (Pin_3), J6.3 (Pin_3)
- net at R8.1, RV4.3: no longer RV4.0 (ShieldPin)
- net at R6.1, RV3.3: no longer RV3.0 (ShieldPin)

Commit message: AttVert pre-jlc
Parts:
- R1, R10, R11, R12, R13, R14, R18, R2, R20, R3, R4, R9: LCSC C14675 -> C25803
- R15, R16, R17, R19, R5, R6, R7, R8: LCSC C2907002 -> C21190
- R21, R22: LCSC C2907011 -> C4184
- U2: LCSC C67473 -> C6961
Changed lines of the file:
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@@
       (effects (font (size 1.27 1.27)) hide)
     )
-    (property "LCSC" "C2907011" (id 4) (at 163.83 144.78 0)
+    (property "LCSC" "C4184" (id 4) (at 163.83 144.78 0)
       (effects (font (size 1.27 1.27)) hide)
     )
@@
       (effects (font (size 1.27 1.27)) hide)
     )
-    (property "LCSC" "C2907002" (id 4) (at 127 71.12 0)
+    (property "LCSC" "C21190" (id 4) (at 127 71.12 0)
       (effects (font (size 1.27 1.27)) hide)
     )
@@
       (effects (font (size 1.27 1.27)) hide)
     )
-    (property "LCSC" "C2907002" (id 4) (at 88.9 121.92 0)
+    (property "LCSC" "C21190" (id 4) (at 88.9 121.92 0)
       (effects (font (size 1.27 1.27)) hide)
     )
@@
       (effects (font (size 1.27 1.27)) hide)
     )
-    (property "LCSC" "C14675" (id 4) (at 71.12 48.26 0)
+    (property "LCSC" "C25803" (id 4) (at 71.12 48.26 0)
       (effects (font (size 1.27 1.27)) hide)
     )
@@
       (effects (font (size 1.27 1.27)) hide)
     )
-    (property "LCSC" "C2907002" (id 4) (at 156.21 113.03 0)
+    (property "LCSC" "C21190" (id 4) (at 156.21 113.03 0)
       (effects (font (size 1.27 1.27)) hide)
     )
@@
       (effects (font (size 1.27 1.27)) hide)
     )
-    (property "LCSC" "C2907002" (id 4) (at 156.21 38.1 0)
+    (property "LCSC" "C21190" (id 4) (at 156.21 38.1 0)
       (effects (font (size 1.27 1.27)) hide)
     )
@@
       (effects (font (size 1.27 1.27)) hide)
     )
-    (property "LCSC" "C2907002" (id 4) (at 88.9 46.99 0)
+    (property "LCSC" "C21190" (id 4) (at 88.9 46.99 0)
       (effects (font (size 1.27 1.27)) hide)
     )
@@
       (effects (font (size 1.27 1.27)) hide)
     )
-    (property "LCSC" "C14675" (id 4) (at 96.52 135.89 0)
+    (property "LCSC" "C25803" (id 4) (at 96.52 135.89 0)
       (effects (font (size 1.27 1.27)) hide)
     )
@@
       (effects (font (size 1.27 1.27)) hide)
     )
-    (property "LCSC" "C67473" (id 4) (at 171.45 135.89 0)
+    (property "LCSC" "C6961" (id 4) (at 171.45 135.89 0)
       (effects (font (size 1.27 1.27)) hide)
     )
@@
       (effects (font (size 1.27 1.27)) hide)
     )
-    (property "LCSC" "C2907002" (id 4) (at 127 146.05 0)
+    (property "LCSC" "C21190" (id 4) (at 127 146.05 0)
       (effects (font (size 1.27 1.27)) hide)
     )
@@
       (effects (font (size 1.27 1.27)) hide)
     )
-    (property "LCSC" "C14675" (id 4) (at 156.21 63.5 0)
+    (property "LCSC" "C25803" (id 4) (at 156.21 63.5 0)
       (effects (font (size 1.27 1.27)) hide)
     )
@@
       (effects (font (size 1.27 1.27)) hide)
     )
-    (property "LCSC" "C14675" (id 4) (at 111.76 48.26 0)
+    (property "LCSC" "C25803" (id 4) (at 111.76 48.26 0)
       (effects (font (size 1.27 1.27)) hide)
     )
@@
       (effects (font (size 1.27 1.27)) hide)
     )
-    (property "LCSC" "C2907011" (id 4) (at 163.83 69.85 0)
+    (property "LCSC" "C4184" (id 4) (at 163.83 69.85 0)
       (effects (font (size 1.27 1.27)) hide)
     )
@@
       (effects (font (size 1.27 1.27)) hide)
     )
-    (property "LCSC" "C14675" (id 4) (at 50.8 133.35 0)
+    (property "LCSC" "C25803" (id 4) (at 50.8 133.35 0)
       (effects (font (size 1.27 1.27)) hide)
     )
@@
       (effects (font (size 1.27 1.27)) hide)
     )
-    (property "LCSC" "C14675" (id 4) (at 96.52 110.49 0)
+    (property "LCSC" "C25803" (id 4) (at 96.52 110.49 0)
       (effects (font (size 1.27 1.27)) hide)
     )
@@
       (effects (font (size 1.27 1.27)) hide)
     )
-    (property "LCSC" "C14675" (id 4) (at 96.52 35.56 0)
+    (property "LCSC" "C25803" (id 4) (at 96.52 35.56 0)
       (effects (font (size 1.27 1.27)) hide)
     )
@@
       (effects (font (size 1.27 1.27)) hide)
     )
-    (property "LCSC" "C14675" (id 4) (at 71.12 123.19 0)
+    (property "LCSC" "C25803" (id 4) (at 71.12 123.19 0)
       (effects (font (size 1.27 1.27)) hide)
     )
@@
       (effects (font (size 1.27 1.27)) hide)
     )
-    (property "LCSC" "C2907002" (id 4) (at 88.9 100.33 0)
+    (property "LCSC" "C21190" (id 4) (at 88.9 100.33 0)
       (effects (font (size 1.27 1.27)) hide)
     )
@@
       (effects (font (size 1.27 1.27)) hide)
     )
-    (property "LCSC" "C67473" (id 4) (at 171.45 60.96 0)
+    (property "LCSC" "C6961" (id 4) (at 171.45 60.96 0)
       (effects (font (size 1.27 1.27)) hide)
     )
@@
       (effects (font (size 1.27 1.27)) hide)
     )
-    (property "LCSC" "C14675" (id 4) (at 111.76 123.19 0)
+    (property "LCSC" "C25803" (id 4) (at 111.76 123.19 0)
       (effects (font (size 1.27 1.27)) hide)
     )
@@
       (effects (font (size 1.27 1.27)) hide)
     )
-    (property "LCSC" "C14675" (id 4) (at 96.52 60.96 0)
+    (property "LCSC" "C25803" (id 4) (at 96.52 60.96 0)
       (effects (font (size 1.27 1.27)) hide)
     )
@@
       (effects (font (size 1.27 1.27)) hide)
     )
-    (property "LCSC" "C14675" (id 4) (at 156.21 138.43 0)
+    (property "LCSC" "C25803" (id 4) (at 156.21 138.43 0)
       (effects (font (size 1.27 1.27)) hide)
     )
@@
       (effects (font (size 1.27 1.27)) hide)
     )
-    (property "LCSC" "C67473" (id 4) (at 274.32 60.96 0)
+    (property "LCSC" "C6961" (id 4) (at 274.32 60.96 0)
       (effects (font (size 1.27 1.27)) hide)
     )
@@
       (effects (font (size 1.27 1.27)) hide)
     )
-    (property "LCSC" "C14675" (id 4) (at 50.8 58.42 0)
+    (property "LCSC" "C25803" (id 4) (at 50.8 58.42 0)
       (effects (font (size 1.27 1.27)) hide)
     )
@@
       (effects (font (size 1.27 1.27)) hide)
     )
-    (property "LCSC" "C2907002" (id 4) (at 88.9 26.67 0)
-      (effects (font (size 1.27 1.27)) hide)
-    )
+    (property "LCSC" "C21190" (id 4) (at 88.9 26.67 0)
+      (effects (font (size 1.27 1.27)) hide)
+    )

Commit message: wip pre-redo orientation
Other:
- company: (none) -> Andrey Salomatin / Pedal Markt
- title: (none) -> AttVert
Changed lines of the file:
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@@
 (kicad_sch (version 20211123) (generator eeschema)
   (paper "A4")
+  (title_block
+    (title "AttVert")
+    (date "2024-12-18")
+    (rev "v1rev2")
+    (company "Andrey Salomatin / Pedal Markt")
+  )
   (junction (at 248.92 68.58) (diameter 0) (color 0 0 0 0)
   )
