File: io-board/io-board.kicad_pcb (KiCad board)
At the start: 4 copper layers, 75 x 54 mm, 77 parts, among them J3 Conn, J4 PWR, J5 In, J6 Out, J7 Headphone, J8 Conn, Q1 J201, Q2 3904 BEC, SW1 SignalSW, SW2 PWRSW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

Commit message: wip
Other:
- board text added: "M3"
Changed lines of the file:
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@@
     (pad_to_mask_clearance 0)
     (pcbplotparams
-      (layerselection 0x00010fc_ffffffff)
+      (layerselection 0x00410fc_ffffffff)
       (disableapertmacros false)
       (usegerberextensions false)
@@
       (sketchpadsonfab false)
       (subtractmaskfromsilk false)
-      (outputformat 1)
+      (outputformat 3)
       (mirror false)
-      (drillshape 1)
+      (drillshape 0)
       (scaleselection 1)
-      (outputdirectory "")
+      (outputdirectory "dxf/")
     )
   )
@@
     )
     (fp_line (start 0 -9.3) (end 0 6.5) (layer "F.SilkS") (width 0.12))
-    (fp_line (start 0 6.5) (end -21.5 6.5) (layer "F.SilkS") (width 0.12))
     (fp_line (start -21.5 -9.3) (end 0 -9.3) (layer "F.SilkS") (width 0.12))
+    (fp_line (start 0 6.5) (end -21.5 6.5) (layer "F.SilkS") (width 0.12))
     (fp_line (start -21.5 6.5) (end -21.5 -9.3) (layer "F.SilkS") (width 0.12))
-    (fp_line (start 4.3 7) (end -26.5 7) (layer "F.CrtYd") (width 0.05))
-    (fp_line (start -26.5 -9.8) (end 4.3 -9.8) (layer "F.CrtYd") (width 0.05))
+    (fp_line (start 8 -9.8) (end 8 7) (layer "F.CrtYd") (width 0.05))
+    (fp_line (start -26.5 -9.8) (end 8 -9.8) (layer "F.CrtYd") (width 0.05))
     (fp_line (start -26.5 7) (end -26.5 -9.8) (layer "F.CrtYd") (width 0.05))
-    (fp_line (start 4.3 -9.8) (end 4.3 7) (layer "F.CrtYd") (width 0.05))
-    (fp_line (start 0 3.3) (end 4.3 3.3) (layer "User.1") (width 0.05))
-    (fp_line (start 4.3 3.3) (end 4.3 -3.3) (layer "User.1") (width 0.05))
-    (fp_line (start 4.3 -3.3) (end 0 -3.3) (layer "User.1") (width 0.05))
+    (fp_line (start 8 7) (end -26.5 7) (layer "F.CrtYd") (width 0.05))
+    (fp_line (start -24.7 -4.2) (end -24.7 4.2) (layer "User.1") (width 0.05))
+    (fp_line (start 8 -4.6) (end 0 -4.6) (layer "User.1") (width 0.05))
+    (fp_line (start 8 4.6) (end 8 -4.6) (layer "User.1") (width 0.05))
+    (fp_line (start 0 4.6) (end 8 4.6) (layer "User.1") (width 0.05))
+    (fp_line (start -21.5 -4.2) (end -24.7 -4.2) (layer "User.1") (width 0.05))
+    (fp_line (start -24.7 4.2) (end -21.5 4.2) (layer "User.1") (width 0.05))
     (pad "R" thru_hole circle locked (at -10.5 -6.9 90) (size 3.2 3.2) (drill 1.6) (layers *.Cu *.Mask)
       (net 23 "unconnected-(J6-PadR)") (pintype "passive+no_connect"))
@@
     (fp_line (start 1 0.6) (end 1 -0.6) (layer "F.Fab") (width 0.1))
     (fp_line (start -1 -0.3) (end -1 0.6) (layer "F.Fab") (width 0.1))
-    (pad "1" smd roundrect (at -1.025 0 180) (size 1.15 1.4) (layers "F.Cu" "F.Paste" "F.Mask") (roundrect_rratio 0.217391)
+    (pad "1" smd roundrect (at -1.025 0 180) (size 1.15 1.4) (layers "F.Cu" "F.Paste" "F.Mask") (roundrect_rratio 0.2173913043)
       (net 17 "Net-(D1-Pad1)") (pinfunction "K") (pintype "passive"))
-    (pad "2" smd roundrect (at 1.025 0 180) (size 1.15 1.4) (layers "F.Cu" "F.Paste" "F.Mask") (roundrect_rratio 0.217391)
+    (pad "2" smd roundrect (at 1.025 0 180) (size 1.15 1.4) (layers "F.Cu" "F.Paste" "F.Mask") (roundrect_rratio 0.2173913043)
       (net 5 "/Von") (pinfunction "A") (pintype "passive"))
     (model "${KICAD6_3DMODEL_DIR}/LED_SMD.3dshapes/LED_0805_2012Metric.wrl"
@@
       (effects (font (size 1 1) (thickness 0.15)))
     )
+    (fp_line (start -21.5 -9.3) (end 0 -9.3) (layer "F.SilkS") (width 0.12))
     (fp_line (start -21.5 6.5) (end -21.5 -9.3) (layer "F.SilkS") (width 0.12))
     (fp_line (start 0 6.5) (end -21.5 6.5) (layer "F.SilkS") (width 0.12))
-    (fp_line (start -21.5 -9.3) (end 0 -9.3) (layer "F.SilkS") (width 0.12))
     (fp_line (start 0 -9.3) (end 0 6.5) (layer "F.SilkS") (width 0.12))
-    (fp_line (start 4.3 -9.8) (end 4.3 7) (layer "F.CrtYd") (width 0.05))
-    (fp_line (start 4.3 7) (end -26.5 7) (layer "F.CrtYd") (width 0.05))
-    (fp_line (start -26.5 -9.8) (end 4.3 -9.8) (layer "F.CrtYd") (width 0.05))
+    (fp_line (start 8 -9.8) (end 8 7) (layer "F.CrtYd") (width 0.05))
     (fp_line (start -26.5 7) (end -26.5 -9.8) (layer "F.CrtYd") (width 0.05))
-    (fp_line (start 4.3 3.3) (end 4.3 -3.3) (layer "User.1") (width 0.05))
-    (fp_line (start 0 3.3) (end 4.3 3.3) (layer "User.1") (width 0.05))
-    (fp_line (start 4.3 -3.3) (end 0 -3.3) (layer "User.1") (width 0.05))
+    (fp_line (start 8 7) (end -26.5 7) (layer "F.CrtYd") (width 0.05))
+    (fp_line (start -26.5 -9.8) (end 8 -9.8) (layer "F.CrtYd") (width 0.05))
+    (fp_line (start -21.5 -4.2) (end -24.7 -4.2) (layer "User.1") (width 0.05))
+    (fp_line (start -24.7 -4.2) (end -24.7 4.2) (layer "User.1") (width 0.05))
+    (fp_line (start -24.7 4.2) (end -21.5 4.2) (layer "User.1") (width 0.05))
+    (fp_line (start 8 -4.6) (end 0 -4.6) (layer "User.1") (width 0.05))
+    (fp_line (start 0 4.6) (end 8 4.6) (layer "User.1") (width 0.05))
+    (fp_line (start 8 4.6) (end 8 -4.6) (layer "User.1") (width 0.05))
     (pad "R" thru_hole circle locked (at -10.5 -6.9 90) (size 3.2 3.2) (drill 1.6) (layers *.Cu *.Mask)
       (net 20 "unconnected-(J5-PadR)") (pintype "passive+no_connect"))
@@
   (gr_arc (start 60 63) (mid 60.87868 60.87868) (end 63 60) (layer "Edge.Cuts") (width 0.1))
   (gr_line (start 135 63) (end 135 111) (layer "Edge.Cuts") (width 0.1))
+  (gr_line (start 57 117) (end 60 117) (layer "User.1") (width 0.15))
+  (gr_line (start 60 117) (end 64.1 110) (layer "User.1") (width 0.15))
   (gr_rect (start 62 62) (end 133 112) (layer "User.2") (width 0.15) (fill none))
+  (gr_text "M3" (at 58.6 115.9) (layer "User.1")
+    (effects (font (size 1 1) (thickness 0.15)))
+  )
+  (dimension (type aligned) (layer "User.1")
+    (pts (xy 116.4 59.9) (xy 135 59.9))
+    (height -17)
+    (gr_text "18.60 mm" (at 125.7 41.75) (layer "User.1")
+      (effects (font (size 1 1) (thickness 0.15)))
+    )
+    (format (units 3) (units_format 1) (precision 2))
+    (style (thickness 0.15) (arrow_length 1.27) (text_position_mode 0) (extension_height 0.58642) (extension_offset 0.5) keep_text_aligned)
+  )
+  (dimension (type aligned) (layer "User.1")
+    (pts (xy 94.5 115.8) (xy 94.5 114))
+    (height -1.4)
+    (gr_text "1.80 mm" (at 91.5 118.5 90) (layer "User.1")
+      (effects (font (size 1 1) (thickness 0.15)))
+    )
+    (format (units 3) (units_format 1) (precision 2))
+    (style (thickness 0.15) (arrow_length 0.4) (text_position_mode 2) (extension_height 0.58642) (extension_offset 0.5) keep_text_aligned)
+  )
+  (dimension (type aligned) (layer "User.1")
+    (pts (xy 97.5 60) (xy 135 60))
+    (height -21.5)
+    (gr_text "37.50 mm" (at 116.25 37.35) (layer "User.1")
+      (effects (font (size 1 1) (thickness 0.15)))
+    )
+    (format (units 3) (units_format 1) (precision 2))
+    (style (thickness 0.15) (arrow_length 1.27) (text_position_mode 0) (extension_height 0.58642) (extension_offset 0.5) keep_text_aligned)
+  )
   (dimension (type aligned) (layer "User.1")
     (pts (xy 60 63) (xy 135 63))
-    (height -15)
-    (gr_text "75.0 mm" (at 97.5 46.85) (layer "User.1")
+    (height -30.5)
+    (gr_text "75.0 mm" (at 97.5 31.35) (layer "User.1")
+      (effects (font (size 1 1) (thickness 0.15)))
+    )
+    (format (units 3) (units_format 1) (precision 1))
+    (style (thickness 0.15) (arrow_length 1.27) (text_position_mode 0) (extension_height 0.58642) (extension_offset 0.5) keep_text_aligned)
+  )
+  (dimension (type aligned) (layer "User.1")
+    (pts (xy 131 110) (xy 131 114))
+    (height -9.5)
+    (gr_text "4.0 mm" (at 139.35 112 90) (layer "User.1")
+      (effects (font (size 1 1) (thickness 0.15)))
+    )
+    (format (units 3) (units_format 1) (precision 1))
+    (style (thickness 0.15) (arrow_length 1.27) (text_position_mode 0) (extension_height 0.58642) (extension_offset 0.5) keep_text_aligned)
+  )
+  (dimension (type aligned) (layer "User.1")
+    (pts (xy 97.5 60) (xy 60 60))
+    (height 21.5)
+    (gr_text "37.50 mm" (at 78.75 37.35) (layer "User.1")
+      (effects (font (size 1 1) (thickness 0.15)))
+    )
+    (format (units 3) (units_format 1) (precision 2))
+    (style (thickness 0.15) (arrow_length 1.27) (text_position_mode 0) (extension_height 0.58642) (extension_offset 0.5) keep_text_aligned)
+  )
+  (dimension (type aligned) (layer "User.1")
+    (pts (xy 102.1 60) (xy 102.1 56.55))
+    (height 3)
+    (gr_text "3.45 mm" (at 104.3 52.7 90) (layer "User.1")
+      (effects (font (size 1 1) (thickness 0.15)))
+    )
+    (format (units 3) (units_format 1) (precision 2))
+    (style (thickness 0.15) (arrow_length 1.27) (text_position_mode 2) (extension_height 0.58642) (extension_offset 0.5) keep_text_aligned)
+  )
+  (dimension (type aligned) (layer "User.1")
+    (pts (xy 121 59.9) (xy 121 51.9))
+    (height 4.3)
+    (gr_text "8.0 mm" (at 124.15 55.9 90) (layer "User.1")
       (effects (font (size 1 1) (thickness 0.15)))
     )
@@
     (style (thickness 0.1) (arrow_length 1.27) (text_position_mode 0) (extension_height 0.58642) (extension_offset 0.5) keep_text_aligned)
   )
+  (dimension (type aligned) (layer "User.1")
+    (pts (xy 81.4 59.9) (xy 60 59.9))
+    (height 17.1)
+    (gr_text "21.40 mm" (at 70.7 41.65) (layer "User.1")
+      (effects (font (size 1 1) (thickness 0.15)))
+    )
+    (format (units 3) (units_format 1) (precision 2))
+    (style (thickness 0.15) (arrow_length 1.27) (text_position_mode 0) (extension_height 0.58642) (extension_offset 0.5) keep_text_aligned)
+  )
   (segment (start 78.9225 79.5815) (end 78.288 78.947) (width 0.5) (layer "B.Cu") (net 1))

Commit message: io jlc part numbers
Parts:
- C10: value 470u -> 10u
- R20, R21, R22, R23: value 1K -> 1R
