File: io-board/io-board.kicad_pcb (KiCad board)
At the start: 4 copper layers, 75 x 54 mm, 77 parts, among them J3 Conn, J4 PWR, J5 In, J6 Out, J7 Headphone, J8 Conn, Q1 J201, Q2 3904 BEC, SW1 SignalSW, SW2 PWRSW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

Commit message: Add jlc num to io board
Other:
- board text added: "JLCJLCJLCJLC"
Changed lines of the file:
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@@
   (gr_line (start 60 117) (end 64.1 110) (layer "User.1") (width 0.15))
   (gr_rect (start 62 62) (end 133 112) (layer "User.2") (width 0.15) (fill none))
+  (gr_text "JLCJLCJLCJLC" (at 97.282 90.678 -270) (layer "B.SilkS")
+    (effects (font (size 0.8 0.8) (thickness 0.15)) (justify mirror))
+  )
   (gr_text "M3" (at 58.6 115.9) (layer "User.1")
     (effects (font (size 1 1) (thickness 0.15)))

Commit message: wip
Parts:
- removed kibuzzard-65D0BA3D: G***, kibuzzard-65D0BA3D
- removed kibuzzard-65D61F93: G***, kibuzzard-65D61F93
- removed kibuzzard-65D61F98 (x2): G***, kibuzzard-65D61F98
- removed kibuzzard-65D62017: G***, kibuzzard-65D62017
- removed kibuzzard-65D62054: G***, kibuzzard-65D62054
- removed kibuzzard-65D621E9: G***, kibuzzard-65D621E9
- removed kibuzzard-65D621F1: G***, kibuzzard-65D621F1
- removed kibuzzard-65D621FF: G***, kibuzzard-65D621FF
- removed kibuzzard-65D6221F: G***, kibuzzard-65D6221F
- removed kibuzzard-65D6222D: G***, kibuzzard-65D6222D
- removed kibuzzard-65D6223E: G***, kibuzzard-65D6223E
- removed kibuzzard-65DA3308: G***, kibuzzard-65DA3308
- added kibuzzard-672CB029: G***, kibuzzard-672CB029, F.Cu at (132.2, 80.7)
- added kibuzzard-672CB033: G***, kibuzzard-672CB033, F.Cu at (132.3, 83.2)
- added kibuzzard-672CB03D: G***, kibuzzard-672CB03D, F.Cu at (132.3, 85.8)
- added kibuzzard-672CB045: G***, kibuzzard-672CB045, F.Cu at (132.3, 88.3)
- added kibuzzard-672CB052: G***, kibuzzard-672CB052, F.Cu at (132.3, 90.9)
- added kibuzzard-672CB05C: G***, kibuzzard-672CB05C, F.Cu at (132.3, 93.4)
- added kibuzzard-672CB0D7: G***, kibuzzard-672CB0D7, F.Cu at (62.6, 83.2)
- added kibuzzard-672CB0E4: G***, kibuzzard-672CB0E4, F.Cu at (62.6, 85.8)
- added kibuzzard-672CB0EB: G***, kibuzzard-672CB0EB, F.Cu at (62.6, 88.3)
- added kibuzzard-672CB0F3: G***, kibuzzard-672CB0F3, F.Cu at (62.6, 90.9)
- added kibuzzard-672CB0F8: G***, kibuzzard-672CB0F8, F.Cu at (62.6, 93.4)
- added kibuzzard-672CB126: G***, kibuzzard-672CB126, F.Cu at (62.6, 80.7)
- added kibuzzard-672CB16D: G***, kibuzzard-672CB16D, B.Cu at (65.3, 101.2)
- D1: footprint LED_SMD:LED_0805_2012Metric_Pad1.15x1.40mm_HandSolder -> LED_SMD:LED_1206_3216Metric_Pad1.42x1.75mm_HandSolder
- R1: value 2.2K -> 4.7K
- U1: value TL072 -> LM358
- moved D1 0.10 mm to (97.6, 77.0)
