File: io-board/headphone.kicad_sch (KiCad schematic)
At the start: 0 parts

Commit message: IO Board wip
Parts:
- added C10: 470u, Capacitor_SMD:CP_Elec_4x5.4, symbol Device:C_Polarized
- added C11, C12, C13: 100n, Capacitor_SMD:C_0603_1608Metric_Pad1.08x0.95mm_HandSolder, symbol Device:C_Small
- added C7, C9: 100n, Capacitor_SMD:CP_Elec_4x5.4, symbol Device:C_Polarized
- added C8: 10u, Capacitor_SMD:CP_Elec_4x5.4, symbol Device:C_Polarized
- added R10, R13: 1M, Resistor_SMD:R_0603_1608Metric_Pad0.98x0.95mm_HandSolder, symbol Device:R
- added R11, R12: 10K, Resistor_SMD:R_0603_1608Metric_Pad0.98x0.95mm_HandSolder, symbol Device:R
- added R14: 10, Resistor_SMD:R_0603_1608Metric_Pad0.98x0.95mm_HandSolder, symbol Device:R
- added R15: 4.7K, Resistor_SMD:R_0603_1608Metric_Pad0.98x0.95mm_HandSolder, symbol Device:R
- added R16, R17, R20, R21, R22, R23: 1K, Resistor_SMD:R_0603_1608Metric_Pad0.98x0.95mm_HandSolder, symbol Device:R
- added R18, R19: 2.2K, Resistor_SMD:R_0603_1608Metric_Pad0.98x0.95mm_HandSolder, symbol Device:R
- added RV1: A20K, R0904NB10KL-25KQ:V3_TRIM_R0904NB10KL-Keepout, symbol Pots:R_Potentiometer_Shield
- added U1: TL072, Package_SO:SOIC-8_3.9x4.9mm_P1.27mm, symbol Amplifier_Operational:TL072
- added U2, U3: NE5532, Package_SO:SOIC-8_3.9x4.9mm_P1.27mm, symbol Amplifier_Operational:NE5532
Connections:
- new net: R17.2, R19.1, U3.2 (-)
- new net: C7.1, R13.1, U1.3 (+)
- new net: R15.1, RV1.2, U2.3 (+), U3.3 (+)
- new net: R14.1, U1.6 (-), U1.7
- new net: C9.1, U1.1, U1.2 (-)
- new net: C9.2, RV1.3
- new net: R16.2, R18.1, U2.2 (-)
- new net: R18.2, R21.1, U2.1, U2.5 (+)
- new net: R20.1, U2.6 (-), U2.7
- new net: C8.1, R11.2, R12.1, U1.5 (+)
- new net: R19.2, R23.1, U3.1, U3.5 (+)
- new net: R22.1, U3.6 (-), U3.7
- new net +4.5V: C10.1, R13.2, R14.2, R15.2, R16.1, R17.1, RV1.1
- new net +9V: C11.1, C12.1, C13.1, R11.1, U1.8 (V+), U2.8 (V+), U3.8 (V+)
- new net GND: C10.2, C11.2, C12.2, C13.2, C8.2, R10.2, R12.2, RV1.0 (ShieldPin), U1.4 (V-), U2.4 (V-), U3.4 (V-)
- new net HeadphoneL: R20.2, R21.2
- new net HeadphoneR: R22.2, R23.2
- new net ToHeadphoneAmp: C7.2, R10.1

Commit message: wip
Parts:
- C8: Mouser (none) -> 710-865080340001
Changed lines of the file:
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@@
+      (effects (font (size 1.27 1.27)) hide)
+    )
+    (property "Mouser" "710-865080340001" (id 4) (at 90.17 135.89 0)
       (effects (font (size 1.27 1.27)) hide)
     )

Commit message: wip
Parts:
- C10: value 470u -> 10u
- R20, R21, R22, R23: value 1K -> 1R; LCSC C234360 -> (none)
Changed lines of the file:
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@@
       (effects (font (size 1.27 1.27)) (justify left))
     )
-    (property "Value" "470u" (id 1) (at 138.43 136.2709 0)
+    (property "Value" "10u" (id 1) (at 138.43 136.2709 0)
       (effects (font (size 1.27 1.27)) (justify left))
     )
@@
     (in_bom yes) (on_board yes) (fields_autoplaced)
     (property "Reference" "R23" (id 0) (at 213.36 82.55 90))
-    (property "Value" "1K" (id 1) (at 213.36 85.09 90))
+    (property "Value" "1R" (id 1) (at 213.36 85.09 90))
     (property "Footprint" "Resistor_SMD:R_0603_1608Metric_Pad0.98x0.95mm_HandSolder" (id 2) (at 213.36 90.678 90)
       (effects (font (size 1.27 1.27)) hide)
@@
       (effects (font (size 1.27 1.27)) hide)
     )
-    (property "LCSC" "C234360" (id 4) (at 213.36 88.9 0)
+    (property "LCSC" "" (id 4) (at 213.36 88.9 0)
       (effects (font (size 1.27 1.27)) hide)
     )
@@
     (in_bom yes) (on_board yes) (fields_autoplaced)
     (property "Reference" "R20" (id 0) (at 213.36 34.29 90))
-    (property "Value" "1K" (id 1) (at 213.36 36.83 90))
+    (property "Value" "1R" (id 1) (at 213.36 36.83 90))
     (property "Footprint" "Resistor_SMD:R_0603_1608Metric_Pad0.98x0.95mm_HandSolder" (id 2) (at 213.36 42.418 90)
       (effects (font (size 1.27 1.27)) hide)
@@
       (effects (font (size 1.27 1.27)) hide)
     )
-    (property "LCSC" "C234360" (id 4) (at 213.36 40.64 0)
+    (property "LCSC" "" (id 4) (at 213.36 40.64 0)
       (effects (font (size 1.27 1.27)) hide)
     )
@@
     (in_bom yes) (on_board yes) (fields_autoplaced)
     (property "Reference" "R21" (id 0) (at 213.36 46.99 90))
-    (property "Value" "1K" (id 1) (at 213.36 49.53 90))
+    (property "Value" "1R" (id 1) (at 213.36 49.53 90))
     (property "Footprint" "Resistor_SMD:R_0603_1608Metric_Pad0.98x0.95mm_HandSolder" (id 2) (at 213.36 55.118 90)
       (effects (font (size 1.27 1.27)) hide)
@@
       (effects (font (size 1.27 1.27)) hide)
     )
-    (property "LCSC" "C234360" (id 4) (at 213.36 53.34 0)
+    (property "LCSC" "" (id 4) (at 213.36 53.34 0)
       (effects (font (size 1.27 1.27)) hide)
     )
@@
     (in_bom yes) (on_board yes) (fields_autoplaced)
     (property "Reference" "R22" (id 0) (at 213.36 69.85 90))
-    (property "Value" "1K" (id 1) (at 213.36 72.39 90))
+    (property "Value" "1R" (id 1) (at 213.36 72.39 90))
     (property "Footprint" "Resistor_SMD:R_0603_1608Metric_Pad0.98x0.95mm_HandSolder" (id 2) (at 213.36 77.978 90)
       (effects (font (size 1.27 1.27)) hide)
@@
       (effects (font (size 1.27 1.27)) hide)
     )
-    (property "LCSC" "C234360" (id 4) (at 213.36 76.2 0)
-      (effects (font (size 1.27 1.27)) hide)
-    )
+    (property "LCSC" "" (id 4) (at 213.36 76.2 0)
+      (effects (font (size 1.27 1.27)) hide)
+    )

Commit message: io jlc part numbers
Parts:
- C10, C8: LCSC (none) -> C240540
- C11, C12, C13: LCSC (none) -> C497032
- R10, R13: LCSC C234360 -> C105578
- R11, R12: LCSC C234360 -> C25804
- R14: LCSC C234360 -> C22859
- R15: LCSC C234360 -> C23162
- R16, R17: LCSC C234360 -> C21190
- R18, R19: LCSC C234360 -> C4190
- R20, R21, R22, R23: LCSC (none) -> C22936
- U1: LCSC (none) -> C6961
- U2, U3: LCSC (none) -> C7426
Changed lines of the file:
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@@
       (effects (font (size 1.27 1.27)) hide)
     )
-    (property "LCSC" "C234360" (id 4) (at 157.48 66.04 0)
+    (property "LCSC" "C21190" (id 4) (at 157.48 66.04 0)
       (effects (font (size 1.27 1.27)) hide)
     )
@@
       (effects (font (size 1.27 1.27)) hide)
     )
-    (property "LCSC" "C234360" (id 4) (at 55.88 54.61 0)
+    (property "LCSC" "C105578" (id 4) (at 55.88 54.61 0)
       (effects (font (size 1.27 1.27)) hide)
     )
@@
       (effects (font (size 1.27 1.27)) hide)
     )
+    (property "LCSC" "C497032" (id 4) (at 255.27 139.7 0)
+      (effects (font (size 1.27 1.27)) hide)
+    )
     (pin "1")
     (pin "2")
@@
       (effects (font (size 1.27 1.27)) hide)
     )
-    (property "LCSC" "C234360" (id 4) (at 80.01 54.61 0)
+    (property "LCSC" "C105578" (id 4) (at 80.01 54.61 0)
       (effects (font (size 1.27 1.27)) hide)
     )
@@
       (effects (font (size 1.27 1.27)) hide)
     )
-    (property "LCSC" "C234360" (id 4) (at 134.62 69.85 0)
+    (property "LCSC" "C23162" (id 4) (at 134.62 69.85 0)
       (effects (font (size 1.27 1.27)) hide)
     )
@@
       (effects (font (size 1.27 1.27)) hide)
     )
+    (property "LCSC" "C6961" (id 4) (at 265.43 139.7 0)
+      (effects (font (size 1.27 1.27)) hide)
+    )
     (pin "1")
     (pin "2")
@@
       (effects (font (size 1.27 1.27)) hide)
     )
+    (property "LCSC" "C497032" (id 4) (at 271.78 139.7 0)
+      (effects (font (size 1.27 1.27)) hide)
+    )
     (pin "1")
     (pin "2")
@@
       (effects (font (size 1.27 1.27)) hide)
     )
+    (property "LCSC" "C240540" (id 4) (at 134.62 135.89 0)
+      (effects (font (size 1.27 1.27)) hide)
+    )
     (pin "1")
     (pin "2")
@@
     )
     (property "Datasheet" "http://www.ti.com/lit/ds/symlink/ne5532.pdf" (id 3) (at 246.38 139.7 0)
+      (effects (font (size 1.27 1.27)) hide)
+    )
+    (property "LCSC" "C7426" (id 4) (at 246.38 139.7 0)
       (effects (font (size 1.27 1.27)) hide)
     )
@@
       (effects (font (size 1.27 1.27)) hide)
     )
-    (property "LCSC" "C234360" (id 4) (at 125.73 125.73 0)
+    (property "LCSC" "C22859" (id 4) (at 125.73 125.73 0)
       (effects (font (size 1.27 1.27)) hide)
     )
@@
     )
     (property "Datasheet" "http://www.ti.com/lit/ds/symlink/ne5532.pdf" (id 3) (at 226.06 139.7 0)
+      (effects (font (size 1.27 1.27)) hide)
+    )
+    (property "LCSC" "C7426" (id 4) (at 226.06 139.7 0)
       (effects (font (size 1.27 1.27)) hide)
     )
@@
       (effects (font (size 1.27 1.27)) hide)
     )
-    (property "LCSC" "C234360" (id 4) (at 171.45 27.94 0)
+    (property "LCSC" "C4190" (id 4) (at 171.45 27.94 0)
       (effects (font (size 1.27 1.27)) hide)
     )
@@
       (effects (font (size 1.27 1.27)) hide)
     )
+    (property "LCSC" "C7426" (id 4) (at 198.12 40.64 0)
+      (effects (font (size 1.27 1.27)) hide)
+    )
     (pin "1")
     (pin "2")
@@
       (effects (font (size 1.27 1.27)) hide)
     )
-    (property "LCSC" "C234360" (id 4) (at 78.74 135.89 0)
+    (property "LCSC" "C25804" (id 4) (at 78.74 135.89 0)
       (effects (font (size 1.27 1.27)) hide)
     )
@@
       (effects (font (size 1.27 1.27)) hide)
     )
-    (property "LCSC" "" (id 4) (at 213.36 88.9 0)
+    (property "LCSC" "C22936" (id 4) (at 213.36 88.9 0)
       (effects (font (size 1.27 1.27)) hide)
     )
@@
       (effects (font (size 1.27 1.27)) hide)
     )
+    (property "LCSC" "C7426" (id 4) (at 171.45 43.18 0)
+      (effects (font (size 1.27 1.27)) hide)
+    )
     (pin "1")
     (pin "2")
@@
       (effects (font (size 1.27 1.27)) hide)
     )
-    (property "LCSC" "C234360" (id 4) (at 157.48 27.94 0)
+    (property "LCSC" "C21190" (id 4) (at 157.48 27.94 0)
       (effects (font (size 1.27 1.27)) hide)
     )
@@
       (effects (font (size 1.27 1.27)) hide)
     )
+    (property "LCSC" "C6961" (id 4) (at 106.68 48.26 0)
+      (effects (font (size 1.27 1.27)) hide)
+    )
     (pin "1")
     (pin "2")
@@
       (effects (font (size 1.27 1.27)) hide)
     )
+    (property "LCSC" "C6961" (id 4) (at 106.68 125.73 0)
+      (effects (font (size 1.27 1.27)) hide)
+    )
     (pin "1")
     (pin "2")
@@
       (effects (font (size 1.27 1.27)) hide)
     )
-    (property "LCSC" "C234360" (id 4) (at 171.45 66.04 0)
+    (property "LCSC" "C4190" (id 4) (at 171.45 66.04 0)
       (effects (font (size 1.27 1.27)) hide)
     )
@@
       (effects (font (size 1.27 1.27)) hide)
     )
-    (property "LCSC" "" (id 4) (at 213.36 40.64 0)
+    (property "LCSC" "C22936" (id 4) (at 213.36 40.64 0)
       (effects (font (size 1.27 1.27)) hide)
     )
@@
       (effects (font (size 1.27 1.27)) hide)
     )
-    (property "LCSC" "C234360" (id 4) (at 78.74 120.65 0)
+    (property "LCSC" "C25804" (id 4) (at 78.74 120.65 0)
       (effects (font (size 1.27 1.27)) hide)
     )
@@
     )
     (property "Mouser" "710-865080340001" (id 4) (at 90.17 135.89 0)
+      (effects (font (size 1.27 1.27)) hide)
+    )
+    (property "LCSC" "C240540" (id 5) (at 90.17 135.89 0)
       (effects (font (size 1.27 1.27)) hide)
     )
@@
       (effects (font (size 1.27 1.27)) hide)
     )
+    (property "LCSC" "C7426" (id 4) (at 171.45 78.74 0)
+      (effects (font (size 1.27 1.27)) hide)
+    )
     (pin "1")
     (pin "2")
@@
       (effects (font (size 1.27 1.27)) hide)
     )
+    (property "LCSC" "C7426" (id 4) (at 198.12 76.2 0)
+      (effects (font (size 1.27 1.27)) hide)
+    )
     (pin "1")
     (pin "2")
@@
       (effects (font (size 1.27 1.27)) hide)
     )
-    (property "LCSC" "" (id 4) (at 213.36 53.34 0)
+    (property "LCSC" "C22936" (id 4) (at 213.36 53.34 0)
       (effects (font (size 1.27 1.27)) hide)
     )
@@
     )
     (property "Datasheet" "~" (id 3) (at 234.95 139.7 0)
+      (effects (font (size 1.27 1.27)) hide)
+    )
+    (property "LCSC" "C497032" (id 4) (at 234.95 139.7 0)
       (effects (font (size 1.27 1.27)) hide)
     )
@@
       (effects (font (size 1.27 1.27)) hide)
     )
-    (property "LCSC" "" (id 4) (at 213.36 76.2 0)
-      (effects (font (size 1.27 1.27)) hide)
-    )
+    (property "LCSC" "C22936" (id 4) (at 213.36 76.2 0)
+      (effects (font (size 1.27 1.27)) hide)
+    )

Commit message: JLC got 100n caps
Parts:
- C7, C9: LCSC (none) -> C271438
Changed lines of the file:
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@@
+      (effects (font (size 1.27 1.27)) hide)
+    )
+    (property "LCSC" "C271438" (id 4) (at 121.92 48.26 0)
       (effects (font (size 1.27 1.27)) hide)
     )
@@
       (effects (font (size 1.27 1.27)) hide)
     )
+    (property "LCSC" "C271438" (id 4) (at 68.58 50.8 0)
+      (effects (font (size 1.27 1.27)) hide)
+    )

Commit message: Protato updates and schem
Other:
- company: (none) -> Andrei Salomatin / Pedal Markt
- title: (none) -> Protato
Changed lines of the file:
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@@
 (kicad_sch (version 20211123) (generator eeschema)
   (paper "A4")
+  (title_block
+    (title "Protato")
+    (rev "v1rev1")
+    (company "Andrei Salomatin / Pedal Markt")
+  )
   (junction (at 179.07 78.74) (diameter 0) (color 0 0 0 0)
   )

Commit message: wip
Parts:
- U1: value TL072 -> NE552; LCSC C6961 -> C7426
Changed lines of the file:
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@@
       (effects (font (size 1.27 1.27)) (justify left))
     )
-    (property "Value" "TL072" (id 1) (at 264.16 140.9699 0)
+    (property "Value" "NE552" (id 1) (at 264.16 140.9699 0)
       (effects (font (size 1.27 1.27)) (justify left))
     )
@@
       (effects (font (size 1.27 1.27)) hide)
     )
-    (property "LCSC" "C6961" (id 4) (at 265.43 139.7 0)
+    (property "LCSC" "C7426" (id 4) (at 265.43 139.7 0)
       (effects (font (size 1.27 1.27)) hide)
     )
@@
     (in_bom yes) (on_board yes) (fields_autoplaced)
     (property "Reference" "U1" (id 0) (at 106.68 38.1 0))
-    (property "Value" "TL072" (id 1) (at 106.68 40.64 0))
+    (property "Value" "NE552" (id 1) (at 106.68 40.64 0))
     (property "Footprint" "Package_SO:SOIC-8_3.9x4.9mm_P1.27mm" (id 2) (at 106.68 48.26 0)
       (effects (font (size 1.27 1.27)) hide)
@@
       (effects (font (size 1.27 1.27)) hide)
     )
-    (property "LCSC" "C6961" (id 4) (at 106.68 48.26 0)
+    (property "LCSC" "C7426" (id 4) (at 106.68 48.26 0)
       (effects (font (size 1.27 1.27)) hide)
     )
@@
     (in_bom yes) (on_board yes) (fields_autoplaced)
     (property "Reference" "U1" (id 0) (at 106.68 115.57 0))
-    (property "Value" "TL072" (id 1) (at 106.68 118.11 0))
+    (property "Value" "NE552" (id 1) (at 106.68 118.11 0))
     (property "Footprint" "Package_SO:SOIC-8_3.9x4.9mm_P1.27mm" (id 2) (at 106.68 125.73 0)
       (effects (font (size 1.27 1.27)) hide)
@@
       (effects (font (size 1.27 1.27)) hide)
     )
-    (property "LCSC" "C6961" (id 4) (at 106.68 125.73 0)
-      (effects (font (size 1.27 1.27)) hide)
-    )
+    (property "LCSC" "C7426" (id 4) (at 106.68 125.73 0)
+      (effects (font (size 1.27 1.27)) hide)
+    )

Commit message: wip
Other:
- note added: "Move R14 into the opamp fb loop"
Changed lines of the file:
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@@
     (stroke (width 0) (type default) (color 0 0 0 0))
+  )
+  (text "Move R14 into the opamp fb loop" (at 118.745 116.205 0)
+    (effects (font (size 1.27 1.27)) (justify left bottom))
   )
   (hierarchical_label "+9V" (shape input) (at 78.74 111.76 90)
