File: io-board/io-board.kicad_sch (KiCad schematic)
At the start: 14 parts, among them J3 Conn, J4 PWR, J5 In, J6 Out, J7 Headphone, J8 Conn, SW1 SignalSW, SW2 PWRSW

Commit message: wip
Parts:
- D1: footprint LED_SMD:LED_0805_2012Metric_Pad1.15x1.40mm_HandSolder -> LED_SMD:LED_1206_3216Metric_Pad1.42x1.75mm_HandSolder
- R1: value 2.2K -> 4.7K; LCSC C4190 -> C23162
Changed lines of the file:
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@@
       (effects (font (size 1.27 1.27)) (justify left))
     )
-    (property "Value" "2.2K" (id 1) (at 215.9 41.9099 0)
+    (property "Value" "4.7K" (id 1) (at 215.9 41.9099 0)
       (effects (font (size 1.27 1.27)) (justify left))
     )
@@
       (effects (font (size 1.27 1.27)) hide)
     )
-    (property "LCSC" "C4190" (id 4) (at 213.36 40.64 0)
+    (property "LCSC" "C23162" (id 4) (at 213.36 40.64 0)
       (effects (font (size 1.27 1.27)) hide)
     )
@@
       (effects (font (size 1.27 1.27)) (justify right))
     )
-    (property "Footprint" "LED_SMD:LED_0805_2012Metric_Pad1.15x1.40mm_HandSolder" (id 2) (at 213.36 30.48 0)
+    (property "Footprint" "LED_SMD:LED_1206_3216Metric_Pad1.42x1.75mm_HandSolder" (id 2) (at 213.36 30.48 0)
       (effects (font (size 1.27 1.27)) hide)
     )
@@
     )
     (path "/feeb30d9-4008-4e40-8871-317e49c53cdb"
-      (reference "D1") (unit 1) (value "PWRLED") (footprint "LED_SMD:LED_0805_2012Metric_Pad1.15x1.40mm_HandSolder")
+      (reference "D1") (unit 1) (value "PWRLED") (footprint "LED_SMD:LED_1206_3216Metric_Pad1.42x1.75mm_HandSolder")
     )
     (path "/bedd26ed-9d21-45bf-9f6a-c0e5d3ec5ec5"
@@
     )
     (path "/15de9d7a-900c-460a-a439-04284730a56b"
-      (reference "R1") (unit 1) (value "2.2K") (footprint "Resistor_SMD:R_0603_1608Metric_Pad0.98x0.95mm_HandSolder")
+      (reference "R1") (unit 1) (value "4.7K") (footprint "Resistor_SMD:R_0603_1608Metric_Pad0.98x0.95mm_HandSolder")
     )
     (path "/3dcf1056-a307-4106-90d9-73251143d1a1/e3cbc328-ad88-49bd-8e94-7ba412469749"
@@
     )
     (path "/138f5238-2466-4b40-8443-8253ffd3dc8e/b2598aea-44b6-40b3-9ac7-3fbe187dc4db"
-      (reference "U1") (unit 1) (value "TL072") (footprint "Package_SO:SOIC-8_3.9x4.9mm_P1.27mm")
+      (reference "U1") (unit 1) (value "NE552") (footprint "Package_SO:SOIC-8_3.9x4.9mm_P1.27mm")
     )
     (path "/138f5238-2466-4b40-8443-8253ffd3dc8e/c1d68c63-e268-4977-8045-3fde58b1cbbb"
-      (reference "U1") (unit 2) (value "TL072") (footprint "Package_SO:SOIC-8_3.9x4.9mm_P1.27mm")
+      (reference "U1") (unit 2) (value "NE552") (footprint "Package_SO:SOIC-8_3.9x4.9mm_P1.27mm")
     )
     (path "/138f5238-2466-4b40-8443-8253ffd3dc8e/3cdc37b8-2b1a-44d0-90d0-3c9be675a4f0"
-      (reference "U1") (unit 3) (value "TL072") (footprint "Package_SO:SOIC-8_3.9x4.9mm_P1.27mm")
+      (reference "U1") (unit 3) (value "NE552") (footprint "Package_SO:SOIC-8_3.9x4.9mm_P1.27mm")
     )
     (path "/138f5238-2466-4b40-8443-8253ffd3dc8e/a437a95b-4848-451e-85c3-ac795aa45aa1"

Commit message: wip
Other:
- note added: "Add reverse polarity protection"
Changed lines of the file:
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@@
     (stroke (width 0) (type default) (color 0 0 0 0))
+  )
+  (text "Add reverse polarity protection" (at 144.78 64.77 0)
+    (effects (font (size 1.27 1.27)) (justify left bottom))
   )
   (label "HeadphoneL" (at 106.68 36.83 0)

Commit message: Add TODOs
Other:
- note added: "Move R14 into the opamp fb loop"
- note added: "TODO:"
Changed lines of the file:
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@@
     (stroke (width 0) (type default) (color 0 0 0 0))
   )
-  (text "Add reverse polarity protection" (at 144.78 64.77 0)
+  (text "TODO:" (at 16.51 179.07 0)
+    (effects (font (size 3.54 3.54)) (justify left bottom))
+  )
+  (text "Move R14 into the opamp fb loop" (at 16.51 186.69 0)
     (effects (font (size 1.27 1.27)) (justify left bottom))
   )
+  (text "Add reverse polarity protection" (at 16.51 184.15 0)
+    (effects (font (size 1.27 1.27)) (justify left bottom))
+  )
