File: filter-board/filter-board.kicad_sch (KiCad schematic)
At the start: 16 parts, among them J1 Conn_01x14_Male, J2 Conn_01x14_Male, U1 TL074

Commit message: Filter board layout
Parts:
- J2: footprint (none) -> Connector_PinHeader_2.54mm:PinHeader_1x14_P2.54mm_Vertical
Connections:
- net +4.5V: now also U1.12 (+); no longer U1.5 (+)
- new net: R4.1, U1.13 (-), U1.14
Changed lines of the file:
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@@
     (pin "1")
   )
-  (symbol (lib_id "Amplifier_Operational:TL074") (at 176.53 83.82 0) (mirror x) (unit 2)
+  (symbol (lib_id "Amplifier_Operational:TL074") (at 176.53 83.82 0) (mirror x) (unit 4)
     (in_bom yes) (on_board yes) (fields_autoplaced)
     (property "Reference" "U1" (id 0) (at 176.53 73.66 0))
@@
       (effects (font (size 1.27 1.27)) (justify right))
     )
-    (property "Footprint" "" (id 2) (at 80.01 91.44 0)
+    (property "Footprint" "Connector_PinHeader_2.54mm:PinHeader_1x14_P2.54mm_Vertical" (id 2) (at 80.01 91.44 0)
       (effects (font (size 1.27 1.27)) hide)
     )
@@
     )
     (path "/c7373592-f4b5-42df-b04e-f93fad84185d"
-      (reference "J2") (unit 1) (value "Conn_01x14_Male") (footprint "")
+      (reference "J2") (unit 1) (value "Conn_01x14_Male") (footprint "Connector_PinHeader_2.54mm:PinHeader_1x14_P2.54mm_Vertical")
     )
     (path "/b5abe6a9-7bed-4133-bcfe-4c721a7d07be"
@@
       (reference "U1") (unit 1) (value "TL074") (footprint "Package_SO:SOIC-14_3.9x8.7mm_P1.27mm")
     )
+    (path "/085918df-72b7-4333-8447-de418b873f7a/c4fd6e35-962d-4a63-8b63-c3baed749756"
+      (reference "U1") (unit 2) (value "TL074") (footprint "Package_SO:SOIC-14_3.9x8.7mm_P1.27mm")
+    )
+    (path "/085918df-72b7-4333-8447-de418b873f7a/c16f2b10-0a91-4dfc-817b-0b651b23ace3"
+      (reference "U1") (unit 3) (value "TL074") (footprint "Package_SO:SOIC-14_3.9x8.7mm_P1.27mm")
+    )
     (path "/1f83af37-6ce0-478a-889a-e6cf1405cbc4"
-      (reference "U1") (unit 2) (value "TL074") (footprint "Package_SO:SOIC-14_3.9x8.7mm_P1.27mm")
-    )
-    (path "/085918df-72b7-4333-8447-de418b873f7a/c4fd6e35-962d-4a63-8b63-c3baed749756"
-      (reference "U1") (unit 3) (value "TL074") (footprint "Package_SO:SOIC-14_3.9x8.7mm_P1.27mm")
-    )
-    (path "/085918df-72b7-4333-8447-de418b873f7a/c16f2b10-0a91-4dfc-817b-0b651b23ace3"
       (reference "U1") (unit 4) (value "TL074") (footprint "Package_SO:SOIC-14_3.9x8.7mm_P1.27mm")
     )
@@
       (reference "U2") (unit 1) (value "TL074") (footprint "Package_SO:SOIC-14_3.9x8.7mm_P1.27mm")
     )
-    (path "/a3791ca5-44e8-4812-bdbe-b50a9712e783/e3eee1b4-ac14-4efb-a54a-8a836a8698ae"
+    (path "/a3791ca5-44e8-4812-bdbe-b50a9712e783/f2ded9a6-638f-4023-81d7-e1576c08ed4d"
       (reference "U2") (unit 2) (value "TL074") (footprint "Package_SO:SOIC-14_3.9x8.7mm_P1.27mm")
     )
@@
       (reference "U2") (unit 3) (value "TL074") (footprint "Package_SO:SOIC-14_3.9x8.7mm_P1.27mm")
     )
-    (path "/a3791ca5-44e8-4812-bdbe-b50a9712e783/f2ded9a6-638f-4023-81d7-e1576c08ed4d"
+    (path "/a3791ca5-44e8-4812-bdbe-b50a9712e783/e3eee1b4-ac14-4efb-a54a-8a836a8698ae"
       (reference "U2") (unit 4) (value "TL074") (footprint "Package_SO:SOIC-14_3.9x8.7mm_P1.27mm")
     )
@@
       (reference "U2") (unit 5) (value "TL074") (footprint "Package_SO:SOIC-14_3.9x8.7mm_P1.27mm")
     )
+    (path "/085918df-72b7-4333-8447-de418b873f7a/c0708f1a-db43-45f0-acd5-f039df2c52da"
+      (reference "U3") (unit 1) (value "TL074") (footprint "Package_SO:SOIC-14_3.9x8.7mm_P1.27mm")
+    )
+    (path "/085918df-72b7-4333-8447-de418b873f7a/81da177b-673f-4dd6-8cf7-e27b67f11e67"
+      (reference "U3") (unit 2) (value "TL074") (footprint "Package_SO:SOIC-14_3.9x8.7mm_P1.27mm")
+    )
+    (path "/085918df-72b7-4333-8447-de418b873f7a/8fcd1e28-b5a1-4c38-a856-67cbe0da524a"
+      (reference "U3") (unit 3) (value "TL074") (footprint "Package_SO:SOIC-14_3.9x8.7mm_P1.27mm")
+    )
     (path "/085918df-72b7-4333-8447-de418b873f7a/eb4ffa87-099a-437e-ad93-5456af427b4d"
-      (reference "U3") (unit 1) (value "TL074") (footprint "Package_SO:SOIC-14_3.9x8.7mm_P1.27mm")
-    )
-    (path "/085918df-72b7-4333-8447-de418b873f7a/8fcd1e28-b5a1-4c38-a856-67cbe0da524a"
-      (reference "U3") (unit 2) (value "TL074") (footprint "Package_SO:SOIC-14_3.9x8.7mm_P1.27mm")
-    )
-    (path "/085918df-72b7-4333-8447-de418b873f7a/81da177b-673f-4dd6-8cf7-e27b67f11e67"
-      (reference "U3") (unit 3) (value "TL074") (footprint "Package_SO:SOIC-14_3.9x8.7mm_P1.27mm")
-    )
-    (path "/085918df-72b7-4333-8447-de418b873f7a/c0708f1a-db43-45f0-acd5-f039df2c52da"
       (reference "U3") (unit 4) (value "TL074") (footprint "Package_SO:SOIC-14_3.9x8.7mm_P1.27mm")
     )
@@
       (reference "U4") (unit 1) (value "SSI2164-Split") (footprint "Package_SO:SOIC-16_3.9x9.9mm_P1.27mm")
     )
-    (path "/085918df-72b7-4333-8447-de418b873f7a/0c77e284-f245-48d7-b471-366d2e2e583d"
+    (path "/085918df-72b7-4333-8447-de418b873f7a/ad18d830-8c9c-4dad-a715-a641e7e0ccb7"
       (reference "U4") (unit 2) (value "SSI2164-Split") (footprint "Package_SO:SOIC-16_3.9x9.9mm_P1.27mm")
     )
@@
       (reference "U4") (unit 3) (value "SSI2164-Split") (footprint "Package_SO:SOIC-16_3.9x9.9mm_P1.27mm")
     )
-    (path "/085918df-72b7-4333-8447-de418b873f7a/ad18d830-8c9c-4dad-a715-a641e7e0ccb7"
+    (path "/085918df-72b7-4333-8447-de418b873f7a/0c77e284-f245-48d7-b471-366d2e2e583d"
       (reference "U4") (unit 4) (value "SSI2164-Split") (footprint "Package_SO:SOIC-16_3.9x9.9mm_P1.27mm")
     )
