File: follower-board/follower-board.kicad_pcb (KiCad board)
At the start: 2 copper layers, 53 parts, among them J1 L, J2 R, U1 TL074, U2 TL074

Commit message: Follower layout done
Parts:
- moved R19 196.4 mm to (58.2, 83.1), turned to -90 degrees
- moved C13 193.0 mm to (56.9, 75.4), turned to 90 degrees
- moved D5 191.1 mm to (55.4, 71.6)
- moved R24 184.2 mm to (67.8, 74.9), turned to 90 degrees
- moved D6 182.3 mm to (55.4, 79.2)
- moved R23 182.2 mm to (66.3, 83.1), turned to 90 degrees
- moved R18 180.4 mm to (54.1, 75.4), turned to -90 degrees
- moved R20 180.3 mm to (60.7, 83.1), turned to -90 degrees
- moved C11 178.8 mm to (67.8, 78.7), turned to -90 degrees
- moved R26 178.1 mm to (63.5, 83.1), turned to -90 degrees
- moved U2 177.9 mm to (62.2, 76.2)
- moved R22 176.1 mm to (70.6, 74.9), turned to 90 degrees
- moved R25 173.4 mm to (67.8, 71.1), turned to 90 degrees
- moved R21 165.4 mm to (70.6, 78.7), turned to -90 degrees
- moved C12 164.3 mm to (70.6, 71.1), turned to 90 degrees
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Routing:
- net /RectifiedOut: track 0.00 -> 61.1 mm, vias 0 -> 1
- net Net-(C11-Pad1): track 0.00 -> 55.7 mm
- net /ThreshIn: track 0.00 -> 46.4 mm
- net /Peak Detector/ThreshLim: track 0.00 -> 34.4 mm
- net /PeakOut: track 0.00 -> 33.5 mm, vias 0 -> 1
- net /In: track 0.00 -> 31.8 mm
- net /FollowerOut: track 0.00 -> 26.7 mm
- net Net-(D1-Pad2): track 0.00 -> 26.4 mm
- net Net-(C3-Pad2): track 0.00 -> 25.4 mm
- net Net-(C9-Pad1): track 0.00 -> 24.5 mm
- net /+9V: track 0.00 -> 20.7 mm, vias 0 -> 3
- net Net-(D3-Pad1): track 0.00 -> 17.7 mm
- net Net-(D3-Pad2): track 0.00 -> 17.1 mm
- net /+4.5V: track 0.00 -> 16.9 mm, vias 0 -> 11
- net Net-(D6-Pad1): track 0.00 -> 15.9 mm
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- added copper zone on B.Cu, net /+4.5V
- added copper zone on F.Cu, net /+9V
- added copper zone on In1.Cu, net /GND
- added copper zone on In2.Cu, net /GND
Other:
- board outline added: 27.9 x 50.8 mm
- copper layers 2 -> 4

Commit message: Pot Adapter v1rev1
Parts:
- added G***: LOGO, LOGO, B.Cu at (62.2, 83.8)
- added REF**: OSHW-Logo2_7.3x6mm_SilkScreen, Symbol:OSHW-Logo2_7.3x6mm_SilkScreen, B.Cu at (62.2, 48.3)
- added kibuzzard-666B0D3F: G***, kibuzzard-666B0D3F, B.Cu at (54.9, 50.8)
- added kibuzzard-666B0D4B: G***, kibuzzard-666B0D4B, B.Cu at (54.9, 68.6)
- added kibuzzard-666B0D4B: G***, kibuzzard-666B0D4B, B.Cu at (54.9, 76.2)
- added kibuzzard-666B0D4B: G***, kibuzzard-666B0D4B, B.Cu at (54.9, 61.0)
- added kibuzzard-666B0D4B: G***, kibuzzard-666B0D4B, B.Cu at (54.9, 53.3)
- added kibuzzard-666B0D54: G***, kibuzzard-666B0D54, B.Cu at (54.9, 55.9)
- added kibuzzard-666B0D65: G***, kibuzzard-666B0D65, B.Cu at (69.6, 50.8)
- added kibuzzard-666B0D69: G***, kibuzzard-666B0D69, B.Cu at (69.6, 61.0)
- added kibuzzard-666B0D69: G***, kibuzzard-666B0D69, B.Cu at (69.6, 68.6)
- added kibuzzard-666B0D69: G***, kibuzzard-666B0D69, B.Cu at (69.6, 53.3)
- added kibuzzard-666B0D69: G***, kibuzzard-666B0D69, B.Cu at (69.6, 76.2)
- added kibuzzard-666B0D6E: G***, kibuzzard-666B0D6E, B.Cu at (69.6, 55.9)
- added kibuzzard-6673DE4D: G***, kibuzzard-6673DE4D, F.Cu at (62.2, 86.6)
- added kibuzzard-6673DFE6: G***, kibuzzard-6673DFE6, B.Cu at (54.9, 58.4)
- added kibuzzard-6673E02E: G***, kibuzzard-6673E02E, B.Cu at (56.9, 66.0)
- added kibuzzard-6673E072: G***, kibuzzard-6673E072, B.Cu at (55.0, 73.7)
- added kibuzzard-6673E097: G***, kibuzzard-6673E097, B.Cu at (69.6, 58.4)
- added kibuzzard-6673E0D0: G***, kibuzzard-6673E0D0, B.Cu at (67.6, 66.0)
- added kibuzzard-6673E113: G***, kibuzzard-6673E113, B.Cu at (55.9, 71.1)
- added kibuzzard-6673E129: G***, kibuzzard-6673E129, B.Cu at (68.5, 71.1)
- added kibuzzard-6673E139: G***, kibuzzard-6673E139, B.Cu at (69.5, 63.5)
- added kibuzzard-6673E150: G***, kibuzzard-6673E150, B.Cu at (55.0, 63.5)
- added kibuzzard-6673E1AC: G***, kibuzzard-6673E1AC, B.Cu at (69.5, 73.7)
- J1, J2: moved to B.Cu
- turned J1 to 180 degrees
- turned J2 to 180 degrees
Other:
- board text added: "JLCJLCJLCJLC"
- board text added: "pedalmarkt.com"
- board text added: "v1rev1"
