File: follower-board/follower-board.kicad_sch (KiCad schematic)
At the start: 6 parts, among them J1 L, J2 R

Commit message: wip
Parts:
- J1, J2: footprint (none) -> Connector_PinHeader_2.54mm:PinHeader_1x11_P2.54mm_Vertical

Commit message: wip pre-redo orientation
Other:
- company: (none) -> Andrey Salomatin / Pedal Markt
- title: (none) -> Demod
Changed lines of the file:
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@@
 (kicad_sch (version 20211123) (generator eeschema)
   (paper "A4")
+  (title_block
+    (title "Demod")
+    (date "2024-12-18")
+    (rev "v1rev1")
+    (company "Andrey Salomatin / Pedal Markt")
+  )
   (junction (at 83.82 60.96) (diameter 0) (color 0 0 0 0)
   )
