File: follower-board/peak.kicad_sch (KiCad schematic)
At the start: 15 parts, among them U2 TL074

Commit message: wip
Parts:
- C11, C12: footprint (none) -> Capacitor_SMD:C_0603_1608Metric_Pad1.08x0.95mm_HandSolder; LCSC (none) -> C376774
- C13: footprint (none) -> Capacitor_SMD:C_0603_1608Metric_Pad1.08x0.95mm_HandSolder; LCSC (none) -> C76711
- D5, D6: footprint (none) -> Diode_SMD:D_SOD-123; LCSC (none) -> C81598
- R18: footprint (none) -> Resistor_SMD:R_0603_1608Metric_Pad0.98x0.95mm_HandSolder; LCSC (none) -> C25804
- R19, R22, R23, R24, R25: footprint (none) -> Resistor_SMD:R_0603_1608Metric_Pad0.98x0.95mm_HandSolder; LCSC (none) -> C25803
- R20: footprint (none) -> Resistor_SMD:R_0603_1608Metric_Pad0.98x0.95mm_HandSolder; LCSC (none) -> C13167
- R21, R26: footprint (none) -> Resistor_SMD:R_0603_1608Metric_Pad0.98x0.95mm_HandSolder; LCSC (none) -> C21190
- U2: footprint (none) -> Package_SO:SOIC-14_3.9x8.7mm_P1.27mm; LCSC (none) -> C6963

Commit message: wip
Other:
- note added: "Change R20 to 10k to avoid loading 4.5V source"
- note added: "Change U2 to R2R opamp due to phase reversal issue"
Changed lines of the file:
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@@
     (stroke (width 0) (type default) (color 0 0 0 0))
+  )
+  (text "Change U2 to R2R opamp due to phase reversal issue"
+    (at 76.2 99.06 0)
+    (effects (font (size 1.27 1.27)) (justify left bottom))
+  )
+  (text "Change R20 to 10k to avoid loading 4.5V source" (at 125.73 132.08 0)
+    (effects (font (size 1.27 1.27)) (justify left bottom))
   )
   (label "ThreshLim" (at 116.84 82.55 180)

Commit message: wip pre-redo orientation
Other:
- company: (none) -> Andrey Salomatin / Pedal Markt
- title: (none) -> Demod
Changed lines of the file:
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@@
 (kicad_sch (version 20211123) (generator eeschema)
   (paper "A4")
+  (title_block
+    (title "Demod")
+    (date "2024-12-18")
+    (rev "v1rev1")
+    (company "Andrey Salomatin / Pedal Markt")
+  )
   (junction (at 148.59 45.72) (diameter 0) (color 0 0 0 0)
   )
