File: follower-board/env-follower.kicad_sch (KiCad schematic)
At the start: 32 parts, among them U1 TL074

Commit message: wip
Parts:
- C1: footprint (none) -> Capacitor_SMD:CP_Elec_5x5.4; LCSC (none) -> C72486
- C10, C6: footprint (none) -> Capacitor_SMD:C_0603_1608Metric_Pad1.08x0.95mm_HandSolder; LCSC (none) -> C76711
- C2, C3, C4: footprint (none) -> Capacitor_SMD:C_0603_1608Metric_Pad1.08x0.95mm_HandSolder; LCSC (none) -> C376774
- C5: footprint (none) -> Capacitor_SMD:C_0603_1608Metric_Pad1.08x0.95mm_HandSolder; LCSC (none) -> C59302
- C7: footprint (none) -> Capacitor_SMD:C_0603_1608Metric_Pad1.08x0.95mm_HandSolder; LCSC (none) -> C1589
- C8, C9: footprint (none) -> Capacitor_SMD:C_0603_1608Metric_Pad1.08x0.95mm_HandSolder; LCSC (none) -> C107073
- D1, D2, D4: footprint (none) -> Diode_SMD:D_SOD-123; LCSC (none) -> C81598
- D3: footprint (none) -> LED_THT:LED_D3.0mm
- R1: footprint (none) -> Resistor_SMD:R_0603_1608Metric_Pad0.98x0.95mm_HandSolder; LCSC (none) -> C25804
- R10: footprint (none) -> Resistor_SMD:R_0603_1608Metric_Pad0.98x0.95mm_HandSolder; LCSC (none) -> C103491
- R11: footprint (none) -> Resistor_SMD:R_0603_1608Metric_Pad0.98x0.95mm_HandSolder; LCSC (none) -> C2759765
- R12: footprint (none) -> Resistor_SMD:R_0603_1608Metric_Pad0.98x0.95mm_HandSolder; LCSC (none) -> C445866
- R13: footprint (none) -> Resistor_SMD:R_0603_1608Metric_Pad0.98x0.95mm_HandSolder; LCSC (none) -> C203213
- R14, R15: footprint (none) -> Resistor_SMD:R_0603_1608Metric_Pad0.98x0.95mm_HandSolder; LCSC (none) -> C21190
- R16, R17, R2, R3, R4, R5, R7: footprint (none) -> Resistor_SMD:R_0603_1608Metric_Pad0.98x0.95mm_HandSolder; LCSC (none) -> C25803
- R6: footprint (none) -> Resistor_SMD:R_0603_1608Metric_Pad0.98x0.95mm_HandSolder; LCSC (none) -> C25808
- R8: footprint (none) -> Resistor_SMD:R_0603_1608Metric_Pad0.98x0.95mm_HandSolder; LCSC (none) -> C13167
- R9: footprint (none) -> Resistor_SMD:R_0603_1608Metric_Pad0.98x0.95mm_HandSolder; LCSC (none) -> C22967
- U1: footprint (none) -> Package_SO:SOIC-14_3.9x8.7mm_P1.27mm; LCSC (none) -> C6963

Commit message: wip
Other:
- note added: "Consider more common resistor values"
Changed lines of the file:
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@@
     (stroke (width 0) (type default) (color 0 0 0 0))
+  )
+  (text "Consider more common resistor values" (at 147.32 57.15 0)
+    (effects (font (size 1.27 1.27)) (justify left bottom))
   )
   (hierarchical_label "GND" (shape input) (at 269.24 50.8 270)

Commit message: wip pre-redo orientation
Other:
- company: (none) -> Andrey Salomatin / Pedal Markt
- title: (none) -> Demod
Changed lines of the file:
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@@
 (kicad_sch (version 20211123) (generator eeschema)
   (paper "A4")
+  (title_block
+    (title "Demod")
+    (date "2024-12-18")
+    (rev "v1rev1")
+    (company "Andrey Salomatin / Pedal Markt")
+  )
   (junction (at 203.2 66.04) (diameter 0) (color 0 0 0 0)
   )

Commit message: wip
Connections:
- net +4.5V: no longer C5.1, C6.1, C7.1, C8.1
- net GND: now also C5.1, C6.1, C7.1, C8.1
Other:
- note added: "Follower output is unipolar Larger or equal to +4.5V"
- note added: "LED Indicator"
- note added: "Volume pot pre-In will act as Sensitivity control"
Changed lines of the file:
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@@
     (stroke (width 0) (type default) (color 0 0 0 0))
+  )
+  (text "LED Indicator" (at 254 71.12 0)
+    (effects (font (size 1.27 1.27)) (justify left bottom))
+  )
+  (text "Follower output is unipolar\nLarger or equal to +4.5V"
+    (at 229.235 54.61 0)
+    (effects (font (size 1.27 1.27)) (justify left bottom))
+  )
+  (text "Volume pot pre-In will act\nas Sensitivity control" (at 20.32 40.64 0)
+    (effects (font (size 1.27 1.27)) (justify left bottom))
   )
   (text "Consider more common resistor values" (at 147.32 57.15 0)
@@
     (effects (font (size 1.27 1.27)) (justify right))
   )
-  (hierarchical_label "+4.5V" (shape input) (at 152.4 82.55 180)
+  (hierarchical_label "GND" (shape input) (at 152.4 82.55 270)
     (effects (font (size 1.27 1.27)) (justify right))
   )
