File: vca-board/vca-board.kicad_pcb (KiCad board)
At the start: 4 copper layers, 27.9 x 63.5 mm, 70 parts, among them J1 Conn_01x18_Male, J2 Conn_01x18_Male, U1 SSI2164-Split, U2 TL074, U3 TL074, U4 TL074

Commit message: VCA board routing done
Routing:
- net /+5.35V_Buf: track 0.00 -> 89.4 mm, vias 0 -> 6
- net /+9V: track 0.00 -> 81.8 mm, vias 0 -> 8
- net /VCA2_Out: track 0.00 -> 48.5 mm
- net /VCA3_Out: track 0.00 -> 47.3 mm
- net /VCA1 Exp/VCA1 CV Processing/VCA1_CV_Biased: track 0.00 -> 47.0 mm, vias 0 -> 2
- net /VCA3 Lin/+2V_Buf: track 0.00 -> 44.5 mm, vias 0 -> 8
- net /VCA1_Out: track 0.00 -> 42.5 mm
- net /VCA3 Lin/VCA3 CV Processing/VCA3_CV_Biased: track 0.00 -> 36.2 mm
- net /VCA2_In: track 0.00 -> 33.9 mm
- net /VCA1_CV: track 0.00 -> 33.2 mm
- net /VCA1_In: track 0.00 -> 32.5 mm
- net /VCA2_CV: track 0.00 -> 32.1 mm
- net /VCA3 Lin/SSI4_Out_Sum_In: track 0.00 -> 29.3 mm, vias 0 -> 2
- net /VCA3_In: track 0.00 -> 28.3 mm, vias 0 -> 1
- net /VCA1 Exp/SSI1_Out_Sum_In: track 0.00 -> 28.1 mm, vias 0 -> 2
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Other:
- board text added: "JLCJLCJLCJLC"

Commit message: wip
Parts:
- added kibuzzard-666B0D3F: G***, kibuzzard-666B0D3F, B.Cu at (54.9, 50.8)
- added kibuzzard-666B0D4B: G***, kibuzzard-666B0D4B, B.Cu at (54.9, 91.4)
- added kibuzzard-666B0D4B: G***, kibuzzard-666B0D4B, B.Cu at (54.9, 71.1)
- added kibuzzard-666B0D4B: G***, kibuzzard-666B0D4B, B.Cu at (54.9, 78.7)
- added kibuzzard-666B0D4B: G***, kibuzzard-666B0D4B, B.Cu at (54.9, 58.4)
- added kibuzzard-666B0D4B: G***, kibuzzard-666B0D4B, B.Cu at (54.9, 83.8)
- added kibuzzard-666B0D4B: G***, kibuzzard-666B0D4B, B.Cu at (54.9, 53.3)
- added kibuzzard-666B0D4B: G***, kibuzzard-666B0D4B, B.Cu at (54.9, 66.0)
- added kibuzzard-666B0D54: G***, kibuzzard-666B0D54, B.Cu at (54.9, 55.9)
- added kibuzzard-666B0D65: G***, kibuzzard-666B0D65, B.Cu at (69.6, 50.8)
- added kibuzzard-666B0D69: G***, kibuzzard-666B0D69, B.Cu at (69.6, 71.1)
- added kibuzzard-666B0D69: G***, kibuzzard-666B0D69, B.Cu at (69.6, 78.7)
- added kibuzzard-666B0D69: G***, kibuzzard-666B0D69, B.Cu at (69.6, 53.3)
- added kibuzzard-666B0D69: G***, kibuzzard-666B0D69, B.Cu at (69.6, 66.0)
- added kibuzzard-666B0D69: G***, kibuzzard-666B0D69, B.Cu at (69.6, 83.8)
- added kibuzzard-666B0D69: G***, kibuzzard-666B0D69, B.Cu at (69.6, 58.4)
- added kibuzzard-666B0D69: G***, kibuzzard-666B0D69, B.Cu at (69.6, 91.4)
- added kibuzzard-666B0D6E: G***, kibuzzard-666B0D6E, B.Cu at (69.6, 55.9)
- added kibuzzard-666B0DD6: G***, kibuzzard-666B0DD6, B.Cu at (54.9, 68.6)
- added kibuzzard-666B0E01: G***, kibuzzard-666B0E01, B.Cu at (69.6, 68.6)
- added kibuzzard-666B0E2E: G***, kibuzzard-666B0E2E, B.Cu at (54.9, 61.0)
- added kibuzzard-666B0E3A: G***, kibuzzard-666B0E3A, B.Cu at (54.9, 63.5)
- added kibuzzard-666B0FB2: G***, kibuzzard-666B0FB2, B.Cu at (54.9, 73.7)
- added kibuzzard-666B0FB7: G***, kibuzzard-666B0FB7, B.Cu at (54.9, 76.2)
- added kibuzzard-666B0FBD: G***, kibuzzard-666B0FBD, B.Cu at (54.9, 81.3)
- added kibuzzard-666B0FCE: G***, kibuzzard-666B0FCE, B.Cu at (54.9, 86.4)
- added kibuzzard-666B0FD4: G***, kibuzzard-666B0FD4, B.Cu at (54.9, 88.9)
- added kibuzzard-666B0FDA: G***, kibuzzard-666B0FDA, B.Cu at (54.9, 94.0)
- added kibuzzard-666B0FF4: G***, kibuzzard-666B0FF4, B.Cu at (69.6, 61.0)
- added kibuzzard-666B0FFF: G***, kibuzzard-666B0FFF, B.Cu at (69.6, 63.5)
- added kibuzzard-666B1051: G***, kibuzzard-666B1051, B.Cu at (69.6, 73.7)
- added kibuzzard-666B1057: G***, kibuzzard-666B1057, B.Cu at (69.6, 76.2)
- added kibuzzard-666B105D: G***, kibuzzard-666B105D, B.Cu at (69.6, 81.3)
- added kibuzzard-666B106F: G***, kibuzzard-666B106F, B.Cu at (69.6, 86.4)
- added kibuzzard-666B1074: G***, kibuzzard-666B1074, B.Cu at (69.6, 88.9)
- added kibuzzard-666B107B: G***, kibuzzard-666B107B, B.Cu at (69.6, 94.0)
Connections:
- J1 pad 10: /GND -> /VCA2_CV
- J1 pad 9: /VCA2_CV -> /GND
- J2 pad 10: /GND -> /VCA2_CV
- J2 pad 9: /VCA2_CV -> /GND
Routing:
- net /VCA2_CV: track 32.1 -> 34.8 mm
Other:
- board text added: "1"
- board text added: "10"
- board text added: "11"
- board text added: "12"
- board text added: "13"
- board text added: "14"
- board text added: "15"
- board text added: "16"
- board text added: "17"
- board text added: "18"
- board text added: "2"
- board text added: "3"
- board text added: "4"
- board text added: "5"
- board text added: "6"
- board text added: "7"
- board text added: "8"
- board text added: "9"

Commit message: Filter board schem done
Parts:
- added G***: LOGO, LOGO, B.Cu at (62.2, 99.1)
- added REF**: OSHW-Logo2_7.3x6mm_SilkScreen, Symbol:OSHW-Logo2_7.3x6mm_SilkScreen, B.Cu at (62.2, 46.2)
- added kibuzzard-666B18FD: G***, kibuzzard-666B18FD, F.Cu at (62.2, 99.1)
- C1, C11, C3, C7: value 1n -> 1.2n
- moved R10 6.19 mm to (62.2, 102.6)
Routing:
- net Net-(C4-Pad1): track 7.73 -> 16.9 mm
- net /VCA3_Out: track 47.3 -> 42.7 mm
Other:
- board text added: "pedalmarkt.com"

Commit message: Filter board layout done
Changed lines of the file:
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@@
       ) (layer "B.SilkS") (width 0) (fill solid))
   )
+  (gr_circle (center 50.8 71.12) (end 51.8 71.12) (layer "F.SilkS") (width 0.12) (fill none))
+  (gr_circle (center 73.66 71.12) (end 74.66 71.12) (layer "F.SilkS") (width 0.12) (fill none))
+  (gr_circle (center 73.66 91.44) (end 74.66 91.44) (layer "F.SilkS") (width 0.12) (fill none))
+  (gr_circle (center 50.8 91.44) (end 51.8 91.44) (layer "F.SilkS") (width 0.12) (fill none))
+  (gr_circle (center 73.66 83.82) (end 74.66 83.82) (layer "F.SilkS") (width 0.12) (fill none))
+  (gr_circle (center 73.676 58.42) (end 74.676 58.42) (layer "F.SilkS") (width 0.12) (fill none))
+  (gr_circle (center 73.66 53.34) (end 74.66 53.34) (layer "F.SilkS") (width 0.12) (fill none))
+  (gr_circle (center 50.8 83.82) (end 51.8 83.82) (layer "F.SilkS") (width 0.12) (fill none))
+  (gr_circle (center 50.816 66.04) (end 51.816 66.04) (layer "F.SilkS") (width 0.12) (fill none))
+  (gr_circle (center 73.676 66.04) (end 74.676 66.04) (layer "F.SilkS") (width 0.12) (fill none))
+  (gr_circle (center 50.816 58.42) (end 51.816 58.42) (layer "F.SilkS") (width 0.12) (fill none))
+  (gr_circle (center 73.66 78.74) (end 74.66 78.74) (layer "F.SilkS") (width 0.12) (fill none))
+  (gr_circle (center 50.8 78.74) (end 51.8 78.74) (layer "F.SilkS") (width 0.12) (fill none))
+  (gr_circle (center 50.8 53.34) (end 51.8 53.34) (layer "F.SilkS") (width 0.12) (fill none))
   (gr_arc (start 71.12 40.64) (mid 74.712102 42.127898) (end 76.2 45.72) (layer "Edge.Cuts") (width 0.1))
   (gr_arc (start 53.34 104.14) (mid 49.747898 102.652102) (end 48.26 99.06) (layer "Edge.Cuts") (width 0.1))

Commit message: Pot Adapter v1rev1
Parts:
- J1, J2: moved to B.Cu
- turned J1 to 180 degrees
- turned J2 to 180 degrees
Other:
- board text added: "v1rev1"
