File: vca-board/vca-board.kicad_pcb (KiCad board)
At the start: 4 copper layers, 27.9 x 63.5 mm, 109 parts, among them J1 Conn_01x18_Male, J2 Conn_01x18_Male, U1 SSI2164-Split, U2 TL074, U3 TL074, U4 TL074

Commit message: Remove D from linear VCA + update graphics
Parts:
- removed D2: 1N4148, Diode_SMD:D_SOD-123
- removed kibuzzard-666B0D3F: G***, kibuzzard-666B0D3F
- removed kibuzzard-666B0D4B (x7): G***, kibuzzard-666B0D4B
- removed kibuzzard-666B0D54: G***, kibuzzard-666B0D54
- removed kibuzzard-666B0D65: G***, kibuzzard-666B0D65
- removed kibuzzard-666B0D69 (x7): G***, kibuzzard-666B0D69
- removed kibuzzard-666B0D6E: G***, kibuzzard-666B0D6E
- removed kibuzzard-666B0DD6: G***, kibuzzard-666B0DD6
- removed kibuzzard-666B0E01: G***, kibuzzard-666B0E01
- removed kibuzzard-666B0E2E: G***, kibuzzard-666B0E2E
- removed kibuzzard-666B0E3A: G***, kibuzzard-666B0E3A
- removed kibuzzard-666B0FB2: G***, kibuzzard-666B0FB2
- removed kibuzzard-666B0FB7: G***, kibuzzard-666B0FB7
- removed kibuzzard-666B0FBD: G***, kibuzzard-666B0FBD
- removed kibuzzard-666B0FCE: G***, kibuzzard-666B0FCE
- removed kibuzzard-666B0FD4: G***, kibuzzard-666B0FD4
- removed kibuzzard-666B0FDA: G***, kibuzzard-666B0FDA
- removed kibuzzard-666B0FF4: G***, kibuzzard-666B0FF4
- removed kibuzzard-666B0FFF: G***, kibuzzard-666B0FFF
- removed kibuzzard-666B1051: G***, kibuzzard-666B1051
- removed kibuzzard-666B1057: G***, kibuzzard-666B1057
- removed kibuzzard-666B105D: G***, kibuzzard-666B105D
- removed kibuzzard-666B106F: G***, kibuzzard-666B106F
- removed kibuzzard-666B1074: G***, kibuzzard-666B1074
- removed kibuzzard-666B107B: G***, kibuzzard-666B107B
- added kibuzzard-672CA102: G***, kibuzzard-672CA102, B.Cu at (69.0, 50.8)
- added kibuzzard-672CA109: G***, kibuzzard-672CA109, B.Cu at (69.0, 53.3)
- added kibuzzard-672CA10D: G***, kibuzzard-672CA10D, B.Cu at (69.0, 55.9)
- added kibuzzard-672CA113: G***, kibuzzard-672CA113, B.Cu at (69.0, 58.4)
- added kibuzzard-672CA118: G***, kibuzzard-672CA118, B.Cu at (69.0, 61.0)
- added kibuzzard-672CA11C: G***, kibuzzard-672CA11C, B.Cu at (69.0, 63.5)
- added kibuzzard-672CA121: G***, kibuzzard-672CA121, B.Cu at (69.0, 66.0)
- added kibuzzard-672CA129: G***, kibuzzard-672CA129, B.Cu at (69.2, 68.6)
- added kibuzzard-672CA12F: G***, kibuzzard-672CA12F, B.Cu at (69.0, 71.1)
- added kibuzzard-672CA136: G***, kibuzzard-672CA136, B.Cu at (69.0, 73.7)
- added kibuzzard-672CA13C: G***, kibuzzard-672CA13C, B.Cu at (69.0, 76.2)
- added kibuzzard-672CA140: G***, kibuzzard-672CA140, B.Cu at (69.0, 78.7)
- added kibuzzard-672CA146: G***, kibuzzard-672CA146, B.Cu at (69.2, 81.3)
- added kibuzzard-672CA14B: G***, kibuzzard-672CA14B, B.Cu at (69.0, 83.8)
- added kibuzzard-672CA14F: G***, kibuzzard-672CA14F, B.Cu at (69.0, 86.4)
- added kibuzzard-672CA156: G***, kibuzzard-672CA156, B.Cu at (69.0, 88.9)
- added kibuzzard-672CA15D: G***, kibuzzard-672CA15D, B.Cu at (69.0, 91.4)
- added kibuzzard-672CA162: G***, kibuzzard-672CA162, B.Cu at (69.2, 94.0)
- added kibuzzard-672CA24E: G***, kibuzzard-672CA24E, B.Cu at (55.4, 50.8)
- added kibuzzard-672CA252: G***, kibuzzard-672CA252, B.Cu at (55.4, 53.3)
- added kibuzzard-672CA257: G***, kibuzzard-672CA257, B.Cu at (55.4, 55.9)
- added kibuzzard-672CA25B: G***, kibuzzard-672CA25B, B.Cu at (55.4, 58.4)
- added kibuzzard-672CA260: G***, kibuzzard-672CA260, B.Cu at (55.4, 61.0)
- added kibuzzard-672CA266: G***, kibuzzard-672CA266, B.Cu at (55.4, 63.5)
- added kibuzzard-672CA26A: G***, kibuzzard-672CA26A, B.Cu at (55.4, 66.0)
- added kibuzzard-672CA26E: G***, kibuzzard-672CA26E, B.Cu at (55.2, 68.6)
- added kibuzzard-672CA275: G***, kibuzzard-672CA275, B.Cu at (55.4, 71.1)
- added kibuzzard-672CA27B: G***, kibuzzard-672CA27B, B.Cu at (55.4, 73.7)
- added kibuzzard-672CA280: G***, kibuzzard-672CA280, B.Cu at (55.4, 76.2)
- added kibuzzard-672CA284: G***, kibuzzard-672CA284, B.Cu at (55.4, 78.7)
- added kibuzzard-672CA288: G***, kibuzzard-672CA288, B.Cu at (55.2, 81.3)
- added kibuzzard-672CA28C: G***, kibuzzard-672CA28C, B.Cu at (55.4, 83.8)
- added kibuzzard-672CA293: G***, kibuzzard-672CA293, B.Cu at (55.4, 86.4)
- added kibuzzard-672CA298: G***, kibuzzard-672CA298, B.Cu at (55.4, 88.9)
- added kibuzzard-672CA29D: G***, kibuzzard-672CA29D, B.Cu at (55.4, 91.4)
- added kibuzzard-672CA2A2: G***, kibuzzard-672CA2A2, B.Cu at (55.2, 94.0)
Connections:
- U2 pad 7: Net-(D2-Pad2) -> /VCA3 Lin/VCA3 CV Processing/VCA3_CV_Biased
Routing:
- net /VCA3 Lin/VCA3 CV Processing/VCA3_CV_Biased: track 36.2 -> 28.0 mm
- net Net-(D2-Pad2): track 7.74 -> 0.00 mm
- net Net-(D1-Pad1): track 20.9 -> 18.5 mm
Other:
- board text added: "v1rev2"
- board text removed: "v1rev1"
