File: vca-board/vca3.kicad_sch (KiCad schematic)
At the start: 20 parts, among them U1 SSI2164-Split, U2 TL074, U4 TL074

Commit message: VCA components linked
Parts:
- C1, C3: footprint (none) -> Capacitor_SMD:C_0603_1608Metric_Pad1.08x0.95mm_HandSolder; LCSC (none) -> C3012379
- C16: footprint (none) -> Capacitor_SMD:C_0603_1608Metric_Pad1.08x0.95mm_HandSolder; LCSC (none) -> C76711
- C17: footprint (none) -> Capacitor_Tantalum_SMD:CP_EIA-3216-18_Kemet-A_Pad1.58x1.35mm_HandSolder; LCSC (none) -> C129272
- C2, C4: footprint (none) -> Capacitor_SMD:C_0603_1608Metric_Pad1.08x0.95mm_HandSolder; LCSC (none) -> C160903
- R1: value 10k -> 15k; footprint (none) -> Resistor_SMD:R_0201_0603Metric_Pad0.64x0.40mm_HandSolder; LCSC (none) -> C22809
- R10, R6: LCSC (none) -> C21190
- R2: value 8k -> 12k; footprint (none) -> Resistor_SMD:R_0201_0603Metric_Pad0.64x0.40mm_HandSolder; LCSC (none) -> C22790
- R23: LCSC (none) -> C22859
- R3, R5: footprint (none) -> Resistor_SMD:R_0201_0603Metric_Pad0.64x0.40mm_HandSolder; LCSC (none) -> C25803
- R4, R8: LCSC (none) -> C22962
- R7: LCSC (none) -> C4184
- R9: footprint (none) -> Resistor_SMD:R_0201_0603Metric_Pad0.64x0.40mm_HandSolder; LCSC (none) -> C23352
- U2, U4: footprint (none) -> Package_SO:SOIC-14_3.9x8.7mm_P1.27mm; LCSC (none) -> C6963
Changed lines of the file:
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@@
+      (effects (font (size 1.27 1.27)) hide)
+    )
+    (property "LCSC" "C21190" (id 4) (at 124.46 43.18 0)
       (effects (font (size 1.27 1.27)) hide)
     )
@@
       (effects (font (size 1.27 1.27)) (justify right))
     )
-    (property "Footprint" "" (id 2) (at 138.7348 104.14 0)
+    (property "Footprint" "Capacitor_SMD:C_0603_1608Metric_Pad1.08x0.95mm_HandSolder" (id 2) (at 138.7348 104.14 0)
       (effects (font (size 1.27 1.27)) hide)
     )
     (property "Datasheet" "~" (id 3) (at 139.7 107.95 0)
+      (effects (font (size 1.27 1.27)) hide)
+    )
+    (property "LCSC" "C3012379" (id 4) (at 139.7 107.95 0)
       (effects (font (size 1.27 1.27)) hide)
     )
@@
       (effects (font (size 1.27 1.27)) hide)
     )
+    (property "LCSC" "C22859" (id 4) (at 97.79 144.78 0)
+      (effects (font (size 1.27 1.27)) hide)
+    )
     (pin "1")
     (pin "2")
@@
       (effects (font (size 1.27 1.27)) (justify right))
     )
-    (property "Value" "8k" (id 1) (at 63.5 156.2099 0)
-      (effects (font (size 1.27 1.27)) (justify right))
-    )
-    (property "Footprint" "" (id 2) (at 62.738 154.94 90)
+    (property "Value" "12k" (id 1) (at 63.5 156.2099 0)
+      (effects (font (size 1.27 1.27)) (justify right))
+    )
+    (property "Footprint" "Resistor_SMD:R_0201_0603Metric_Pad0.64x0.40mm_HandSolder" (id 2) (at 62.738 154.94 90)
       (effects (font (size 1.27 1.27)) hide)
     )
     (property "Datasheet" "~" (id 3) (at 60.96 154.94 0)
+      (effects (font (size 1.27 1.27)) hide)
+    )
+    (property "LCSC" "C22790" (id 4) (at 60.96 154.94 0)
       (effects (font (size 1.27 1.27)) hide)
     )
@@
     (property "Reference" "R5" (id 0) (at 88.9 34.29 90))
     (property "Value" "100k" (id 1) (at 88.9 36.83 90))
-    (property "Footprint" "" (id 2) (at 88.9 42.418 90)
+    (property "Footprint" "Resistor_SMD:R_0201_0603Metric_Pad0.64x0.40mm_HandSolder" (id 2) (at 88.9 42.418 90)
       (effects (font (size 1.27 1.27)) hide)
     )
     (property "Datasheet" "~" (id 3) (at 88.9 40.64 0)
+      (effects (font (size 1.27 1.27)) hide)
+    )
+    (property "LCSC" "C25803" (id 4) (at 88.9 40.64 0)
       (effects (font (size 1.27 1.27)) hide)
     )
@@
     (property "Reference" "U2" (id 0) (at 109.22 33.02 0))
     (property "Value" "TL074" (id 1) (at 109.22 35.56 0))
-    (property "Footprint" "" (id 2) (at 107.95 45.72 0)
+    (property "Footprint" "Package_SO:SOIC-14_3.9x8.7mm_P1.27mm" (id 2) (at 107.95 45.72 0)
       (effects (font (size 1.27 1.27)) hide)
     )
     (property "Datasheet" "http://www.ti.com/lit/ds/symlink/tl071.pdf" (id 3) (at 110.49 48.26 0)
+      (effects (font (size 1.27 1.27)) hide)
+    )
+    (property "LCSC" "C6963" (id 4) (at 109.22 43.18 0)
       (effects (font (size 1.27 1.27)) hide)
     )
@@
       (effects (font (size 1.27 1.27)) hide)
     )
+    (property "LCSC" "C22962" (id 4) (at 139.7 99.06 0)
+      (effects (font (size 1.27 1.27)) hide)
+    )
     (pin "1")
     (pin "2")
@@
     (property "Reference" "C4" (id 0) (at 180.34 59.69 90))
     (property "Value" "100p" (id 1) (at 180.34 62.23 90))
-    (property "Footprint" "" (id 2) (at 176.53 68.2752 0)
+    (property "Footprint" "Capacitor_SMD:C_0603_1608Metric_Pad1.08x0.95mm_HandSolder" (id 2) (at 176.53 68.2752 0)
       (effects (font (size 1.27 1.27)) hide)
     )
     (property "Datasheet" "~" (id 3) (at 180.34 67.31 0)
+      (effects (font (size 1.27 1.27)) hide)
+    )
+    (property "LCSC" "C160903" (id 4) (at 180.34 67.31 0)
       (effects (font (size 1.27 1.27)) hide)
     )
@@
     (property "Reference" "U2" (id 0) (at 181.61 82.55 0))
     (property "Value" "TL074" (id 1) (at 181.61 85.09 0))
-    (property "Footprint" "" (id 2) (at 180.34 95.25 0)
+    (property "Footprint" "Package_SO:SOIC-14_3.9x8.7mm_P1.27mm" (id 2) (at 180.34 95.25 0)
       (effects (font (size 1.27 1.27)) hide)
     )
     (property "Datasheet" "http://www.ti.com/lit/ds/symlink/tl071.pdf" (id 3) (at 182.88 97.79 0)
+      (effects (font (size 1.27 1.27)) hide)
+    )
+    (property "LCSC" "C6963" (id 4) (at 181.61 92.71 0)
       (effects (font (size 1.27 1.27)) hide)
     )
@@
       (effects (font (size 1.27 1.27)) hide)
     )
+    (property "LCSC" "C22962" (id 4) (at 60.96 99.06 0)
+      (effects (font (size 1.27 1.27)) hide)
+    )
     (pin "1")
     (pin "2")
@@
     (property "Reference" "C2" (id 0) (at 109.22 20.32 90))
     (property "Value" "100p" (id 1) (at 109.22 22.86 90))
-    (property "Footprint" "" (id 2) (at 113.03 26.9748 0)
+    (property "Footprint" "Capacitor_SMD:C_0603_1608Metric_Pad1.08x0.95mm_HandSolder" (id 2) (at 113.03 26.9748 0)
       (effects (font (size 1.27 1.27)) hide)
     )
     (property "Datasheet" "~" (id 3) (at 109.22 27.94 0)
+      (effects (font (size 1.27 1.27)) hide)
+    )
+    (property "LCSC" "C160903" (id 4) (at 109.22 27.94 0)
       (effects (font (size 1.27 1.27)) hide)
     )
@@
       (effects (font (size 1.27 1.27)) hide)
     )
+    (property "LCSC" "C4184" (id 4) (at 129.54 90.17 0)
+      (effects (font (size 1.27 1.27)) hide)
+    )
     (pin "1")
     (pin "2")
@@
     (property "Reference" "R3" (id 0) (at 54.61 83.82 90))
     (property "Value" "100k" (id 1) (at 54.61 86.36 90))
-    (property "Footprint" "" (id 2) (at 54.61 91.948 90)
+    (property "Footprint" "Resistor_SMD:R_0201_0603Metric_Pad0.64x0.40mm_HandSolder" (id 2) (at 54.61 91.948 90)
       (effects (font (size 1.27 1.27)) hide)
     )
     (property "Datasheet" "~" (id 3) (at 54.61 90.17 0)
+      (effects (font (size 1.27 1.27)) hide)
+    )
+    (property "LCSC" "C25803" (id 4) (at 54.61 90.17 0)
       (effects (font (size 1.27 1.27)) hide)
     )
@@
       (effects (font (size 1.27 1.27)) (justify left))
     )
-    (property "Footprint" "" (id 2) (at 102.5652 158.75 0)
+    (property "Footprint" "Capacitor_Tantalum_SMD:CP_EIA-3216-18_Kemet-A_Pad1.58x1.35mm_HandSolder" (id 2) (at 102.5652 158.75 0)
       (effects (font (size 1.27 1.27)) hide)
     )
@@
       (effects (font (size 1.27 1.27)) hide)
     )
+    (property "LCSC" "C129272" (id 4) (at 101.6 154.94 0)
+      (effects (font (size 1.27 1.27)) hide)
+    )
     (pin "1")
     (pin "2")
@@
       (effects (font (size 1.27 1.27)) (justify right))
     )
-    (property "Footprint" "" (id 2) (at 70.1548 151.13 0)
+    (property "Footprint" "Capacitor_SMD:C_0603_1608Metric_Pad1.08x0.95mm_HandSolder" (id 2) (at 70.1548 151.13 0)
       (effects (font (size 1.27 1.27)) hide)
     )
     (property "Datasheet" "~" (id 3) (at 71.12 154.94 0)
+      (effects (font (size 1.27 1.27)) hide)
+    )
+    (property "LCSC" "C76711" (id 4) (at 71.12 154.94 0)
       (effects (font (size 1.27 1.27)) hide)
     )
@@
     (property "Reference" "R9" (id 0) (at 180.34 72.39 90))
     (property "Value" "24k" (id 1) (at 180.34 74.93 90))
-    (property "Footprint" "" (id 2) (at 180.34 80.518 90)
+    (property "Footprint" "Resistor_SMD:R_0201_0603Metric_Pad0.64x0.40mm_HandSolder" (id 2) (at 180.34 80.518 90)
       (effects (font (size 1.27 1.27)) hide)
     )
@@
       (effects (font (size 1.27 1.27)) hide)
     )
+    (property "LCSC" "C23352" (id 4) (at 180.34 78.74 0)
+      (effects (font (size 1.27 1.27)) hide)
+    )
     (pin "1")
     (pin "2")
@@
       (effects (font (size 1.27 1.27)) (justify right))
     )
-    (property "Footprint" "" (id 2) (at 59.9948 104.14 0)
+    (property "Footprint" "Capacitor_SMD:C_0603_1608Metric_Pad1.08x0.95mm_HandSolder" (id 2) (at 59.9948 104.14 0)
       (effects (font (size 1.27 1.27)) hide)
     )
     (property "Datasheet" "~" (id 3) (at 60.96 107.95 0)
+      (effects (font (size 1.27 1.27)) hide)
+    )
+    (property "LCSC" "C3012379" (id 4) (at 60.96 107.95 0)
       (effects (font (size 1.27 1.27)) hide)
     )
@@
       (effects (font (size 1.27 1.27)) hide)
     )
+    (property "LCSC" "C21190" (id 4) (at 198.12 92.71 0)
+      (effects (font (size 1.27 1.27)) hide)
+    )
     (pin "1")
     (pin "2")
@@
     (property "Reference" "U4" (id 0) (at 83.82 134.62 0))
     (property "Value" "TL074" (id 1) (at 83.82 137.16 0))
-    (property "Footprint" "" (id 2) (at 82.55 147.32 0)
+    (property "Footprint" "Package_SO:SOIC-14_3.9x8.7mm_P1.27mm" (id 2) (at 82.55 147.32 0)
       (effects (font (size 1.27 1.27)) hide)
     )
     (property "Datasheet" "http://www.ti.com/lit/ds/symlink/tl071.pdf" (id 3) (at 85.09 149.86 0)
+      (effects (font (size 1.27 1.27)) hide)
+    )
+    (property "LCSC" "C6963" (id 4) (at 83.82 144.78 0)
       (effects (font (size 1.27 1.27)) hide)
     )
@@
       (effects (font (size 1.27 1.27)) (justify right))
     )
-    (property "Value" "10k" (id 1) (at 63.5 143.5099 0)
-      (effects (font (size 1.27 1.27)) (justify right))
-    )
-    (property "Footprint" "" (id 2) (at 62.738 142.24 90)
+    (property "Value" "15k" (id 1) (at 63.5 143.5099 0)
+      (effects (font (size 1.27 1.27)) (justify right))
+    )
+    (property "Footprint" "Resistor_SMD:R_0201_0603Metric_Pad0.64x0.40mm_HandSolder" (id 2) (at 62.738 142.24 90)
       (effects (font (size 1.27 1.27)) hide)
     )
@@
       (effects (font (size 1.27 1.27)) hide)
     )
+    (property "LCSC" "C22809" (id 4) (at 60.96 142.24 0)
+      (effects (font (size 1.27 1.27)) hide)
+    )

Commit message: VCA board components placed
Parts:
- R1, R2, R3, R5, R9: footprint Resistor_SMD:R_0201_0603Metric_Pad0.64x0.40mm_HandSolder -> Resistor_SMD:R_0603_1608Metric_Pad0.98x0.95mm_HandSolder
- R10, R23, R4, R6, R7, R8: footprint (none) -> Resistor_SMD:R_0603_1608Metric_Pad0.98x0.95mm_HandSolder
- renumbered U4 to U3
Connections:
- net +2V: now also U3.3 (+); no longer U3.12 (+)
- new net: R23.2, U3.1, U3.2 (-)
Changed lines of the file:
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@@
     (property "Reference" "R6" (id 0) (at 124.46 36.83 90))
     (property "Value" "1k" (id 1) (at 124.46 39.37 90))
-    (property "Footprint" "" (id 2) (at 124.46 44.958 90)
+    (property "Footprint" "Resistor_SMD:R_0603_1608Metric_Pad0.98x0.95mm_HandSolder" (id 2) (at 124.46 44.958 90)
       (effects (font (size 1.27 1.27)) hide)
     )
@@
     (property "Reference" "R23" (id 0) (at 97.79 138.43 90))
     (property "Value" "10" (id 1) (at 97.79 140.97 90))
-    (property "Footprint" "" (id 2) (at 97.79 143.002 90)
+    (property "Footprint" "Resistor_SMD:R_0603_1608Metric_Pad0.98x0.95mm_HandSolder" (id 2) (at 97.79 143.002 90)
       (effects (font (size 1.27 1.27)) hide)
     )
@@
       (effects (font (size 1.27 1.27)) (justify right))
     )
-    (property "Footprint" "Resistor_SMD:R_0201_0603Metric_Pad0.64x0.40mm_HandSolder" (id 2) (at 62.738 154.94 90)
+    (property "Footprint" "Resistor_SMD:R_0603_1608Metric_Pad0.98x0.95mm_HandSolder" (id 2) (at 62.738 154.94 90)
       (effects (font (size 1.27 1.27)) hide)
     )
@@
     (property "Reference" "R5" (id 0) (at 88.9 34.29 90))
     (property "Value" "100k" (id 1) (at 88.9 36.83 90))
-    (property "Footprint" "Resistor_SMD:R_0201_0603Metric_Pad0.64x0.40mm_HandSolder" (id 2) (at 88.9 42.418 90)
+    (property "Footprint" "Resistor_SMD:R_0603_1608Metric_Pad0.98x0.95mm_HandSolder" (id 2) (at 88.9 42.418 90)
       (effects (font (size 1.27 1.27)) hide)
     )
@@
       (effects (font (size 1.27 1.27)) (justify right))
     )
-    (property "Footprint" "" (id 2) (at 141.478 99.06 90)
+    (property "Footprint" "Resistor_SMD:R_0603_1608Metric_Pad0.98x0.95mm_HandSolder" (id 2) (at 141.478 99.06 90)
       (effects (font (size 1.27 1.27)) hide)
     )
@@
       (effects (font (size 1.27 1.27)) (justify right))
     )
-    (property "Footprint" "" (id 2) (at 62.738 99.06 90)
+    (property "Footprint" "Resistor_SMD:R_0603_1608Metric_Pad0.98x0.95mm_HandSolder" (id 2) (at 62.738 99.06 90)
       (effects (font (size 1.27 1.27)) hide)
     )
@@
     (property "Reference" "R7" (id 0) (at 129.54 83.82 90))
     (property "Value" "20k" (id 1) (at 129.54 86.36 90))
-    (property "Footprint" "" (id 2) (at 129.54 91.948 90)
+    (property "Footprint" "Resistor_SMD:R_0603_1608Metric_Pad0.98x0.95mm_HandSolder" (id 2) (at 129.54 91.948 90)
       (effects (font (size 1.27 1.27)) hide)
     )
@@
     (property "Reference" "R3" (id 0) (at 54.61 83.82 90))
     (property "Value" "100k" (id 1) (at 54.61 86.36 90))
-    (property "Footprint" "Resistor_SMD:R_0201_0603Metric_Pad0.64x0.40mm_HandSolder" (id 2) (at 54.61 91.948 90)
+    (property "Footprint" "Resistor_SMD:R_0603_1608Metric_Pad0.98x0.95mm_HandSolder" (id 2) (at 54.61 91.948 90)
       (effects (font (size 1.27 1.27)) hide)
     )
@@
     (property "Reference" "R9" (id 0) (at 180.34 72.39 90))
     (property "Value" "24k" (id 1) (at 180.34 74.93 90))
-    (property "Footprint" "Resistor_SMD:R_0201_0603Metric_Pad0.64x0.40mm_HandSolder" (id 2) (at 180.34 80.518 90)
+    (property "Footprint" "Resistor_SMD:R_0603_1608Metric_Pad0.98x0.95mm_HandSolder" (id 2) (at 180.34 80.518 90)
       (effects (font (size 1.27 1.27)) hide)
     )
@@
     (property "Reference" "R10" (id 0) (at 198.12 86.36 90))
     (property "Value" "1k" (id 1) (at 198.12 88.9 90))
-    (property "Footprint" "" (id 2) (at 198.12 94.488 90)
+    (property "Footprint" "Resistor_SMD:R_0603_1608Metric_Pad0.98x0.95mm_HandSolder" (id 2) (at 198.12 94.488 90)
       (effects (font (size 1.27 1.27)) hide)
     )
@@
     (pin "2")
   )
-  (symbol (lib_id "Amplifier_Operational:TL074") (at 83.82 144.78 0) (mirror x) (unit 4)
-    (in_bom yes) (on_board yes) (fields_autoplaced)
-    (property "Reference" "U4" (id 0) (at 83.82 134.62 0))
+  (symbol (lib_id "Amplifier_Operational:TL074") (at 83.82 144.78 0) (mirror x) (unit 1)
+    (in_bom yes) (on_board yes) (fields_autoplaced)
+    (property "Reference" "U3" (id 0) (at 83.82 134.62 0))
     (property "Value" "TL074" (id 1) (at 83.82 137.16 0))
     (property "Footprint" "Package_SO:SOIC-14_3.9x8.7mm_P1.27mm" (id 2) (at 82.55 147.32 0)
@@
       (effects (font (size 1.27 1.27)) (justify right))
     )
-    (property "Footprint" "Resistor_SMD:R_0201_0603Metric_Pad0.64x0.40mm_HandSolder" (id 2) (at 62.738 142.24 90)
-      (effects (font (size 1.27 1.27)) hide)
-    )
+    (property "Footprint" "Resistor_SMD:R_0603_1608Metric_Pad0.98x0.95mm_HandSolder" (id 2) (at 62.738 142.24 90)
+      (effects (font (size 1.27 1.27)) hide)
+    )

Commit message: Filter board schem done
Parts:
- C1, C3: value 1n -> 1.2n; LCSC C3012379 -> C576816
Changed lines of the file:
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@@
       (effects (font (size 1.27 1.27)) (justify right))
     )
-    (property "Value" "1n" (id 1) (at 143.51 109.2199 0)
+    (property "Value" "1.2n" (id 1) (at 143.51 109.2199 0)
       (effects (font (size 1.27 1.27)) (justify right))
     )
@@
       (effects (font (size 1.27 1.27)) hide)
     )
-    (property "LCSC" "C3012379" (id 4) (at 139.7 107.95 0)
+    (property "LCSC" "C576816" (id 4) (at 139.7 107.95 0)
       (effects (font (size 1.27 1.27)) hide)
     )
@@
       (effects (font (size 1.27 1.27)) (justify right))
     )
-    (property "Value" "1n" (id 1) (at 64.77 109.2199 0)
+    (property "Value" "1.2n" (id 1) (at 64.77 109.2199 0)
       (effects (font (size 1.27 1.27)) (justify right))
     )
@@
       (effects (font (size 1.27 1.27)) hide)
     )
-    (property "LCSC" "C3012379" (id 4) (at 60.96 107.95 0)
-      (effects (font (size 1.27 1.27)) hide)
-    )
+    (property "LCSC" "C576816" (id 4) (at 60.96 107.95 0)
+      (effects (font (size 1.27 1.27)) hide)
+    )

Commit message: Remove D from linear VCA + update graphics
Other:
- company: (none) -> Pedal Markt / Andrey Salomatin
- title: (none) -> VCA Board
Changed lines of the file:
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@@
 (kicad_sch (version 20211123) (generator eeschema)
   (paper "A4")
+  (title_block
+    (title "VCA Board")
+    (date "2024-11-07")
+    (rev "v1rev2")
+    (company "Pedal Markt / Andrey Salomatin")
+  )
   (junction (at 139.7 90.17) (diameter 0) (color 0 0 0 0)
   )

Commit message: wip pre-redo orientation
Other:
- company: Pedal Markt / Andrey Salomatin -> Andrey Salomatin / Pedal Markt
- title: VCA Board -> Mag
Changed lines of the file:
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@@
   (paper "A4")
   (title_block
-    (title "VCA Board")
+    (title "Mag")
     (date "2024-11-07")
     (rev "v1rev2")
-    (company "Pedal Markt / Andrey Salomatin")
+    (company "Andrey Salomatin / Pedal Markt")
   )
   (junction (at 139.7 90.17) (diameter 0) (color 0 0 0 0)
