File: lfo-board/lfo-board.kicad_pcb (KiCad board)
At the start: 4 copper layers, 33 x 55.9 mm, 90 parts, among them J1 Conn_01x15, J2 Conn_01x15, Q1 MMBT3904, SW1 SW_Push, U1 MCP6004, U4 StompLFO, U5 L78L05, U6 TL972

Commit message: wip
Parts:
- removed kibuzzard-65FC58C1: G***, kibuzzard-65FC58C1
- removed kibuzzard-65FC5928 (x5): G***, kibuzzard-65FC5928
- removed kibuzzard-65FC593A: G***, kibuzzard-65FC593A
- removed kibuzzard-65FC5990: G***, kibuzzard-65FC5990
- removed kibuzzard-65FC599C: G***, kibuzzard-65FC599C
- removed kibuzzard-65FC59AA: G***, kibuzzard-65FC59AA
- removed kibuzzard-65FC59B5: G***, kibuzzard-65FC59B5
- removed kibuzzard-65FC59D5: G***, kibuzzard-65FC59D5
- removed kibuzzard-65FC59E3: G***, kibuzzard-65FC59E3
- removed kibuzzard-65FC59FD: G***, kibuzzard-65FC59FD
- removed kibuzzard-65FC5A15: G***, kibuzzard-65FC5A15
- removed kibuzzard-65FC5A8F: G***, kibuzzard-65FC5A8F
- removed kibuzzard-65FC5A9B (x5): G***, kibuzzard-65FC5A9B
- removed kibuzzard-65FC5ACC: G***, kibuzzard-65FC5ACC
- removed kibuzzard-65FC5ADA: G***, kibuzzard-65FC5ADA
- removed kibuzzard-65FC5AE2: G***, kibuzzard-65FC5AE2
- removed kibuzzard-65FC5AF0: G***, kibuzzard-65FC5AF0
- removed kibuzzard-65FC5AF9: G***, kibuzzard-65FC5AF9
- removed kibuzzard-65FC5B08: G***, kibuzzard-65FC5B08
- removed kibuzzard-65FC5B16: G***, kibuzzard-65FC5B16
- removed kibuzzard-65FC5B2E: G***, kibuzzard-65FC5B2E
- removed kibuzzard-65FC5B39: G***, kibuzzard-65FC5B39
- added kibuzzard-672CB46D: G***, kibuzzard-672CB46D, B.Cu at (32.4, 58.4)
- added kibuzzard-672CB471: G***, kibuzzard-672CB471, B.Cu at (32.5, 61.0)
- added kibuzzard-672CB474: G***, kibuzzard-672CB474, B.Cu at (32.5, 63.5)
- added kibuzzard-672CB47A: G***, kibuzzard-672CB47A, B.Cu at (31.8, 66.0)
- added kibuzzard-672CB47E: G***, kibuzzard-672CB47E, B.Cu at (32.5, 68.6)
- added kibuzzard-672CB484: G***, kibuzzard-672CB484, B.Cu at (31.8, 71.1)
- added kibuzzard-672CB488: G***, kibuzzard-672CB488, B.Cu at (32.5, 73.7)
- added kibuzzard-672CB48C: G***, kibuzzard-672CB48C, B.Cu at (33.1, 76.2)
- added kibuzzard-672CB496: G***, kibuzzard-672CB496, B.Cu at (32.6, 78.7)
- added kibuzzard-672CB4A3: G***, kibuzzard-672CB4A3, B.Cu at (33.7, 81.3)
- added kibuzzard-672CB4B5: G***, kibuzzard-672CB4B5, B.Cu at (32.5, 83.8)
- added kibuzzard-672CB4C0: G***, kibuzzard-672CB4C0, B.Cu at (32.5, 86.4)
- added kibuzzard-672CB4C9: G***, kibuzzard-672CB4C9, B.Cu at (33.7, 88.9)
- added kibuzzard-672CB4D2: G***, kibuzzard-672CB4D2, B.Cu at (34.3, 91.4)
- added kibuzzard-672CB4D9: G***, kibuzzard-672CB4D9, B.Cu at (32.5, 94.0)
- added kibuzzard-672CB59C: G***, kibuzzard-672CB59C, B.Cu at (51.5, 58.4)
- added kibuzzard-672CB5A6: G***, kibuzzard-672CB5A6, B.Cu at (51.5, 61.0)
- added kibuzzard-672CB5AE: G***, kibuzzard-672CB5AE, B.Cu at (51.5, 63.5)
- added kibuzzard-672CB5B5: G***, kibuzzard-672CB5B5, B.Cu at (52.1, 66.0)
- added kibuzzard-672CB5BD: G***, kibuzzard-672CB5BD, B.Cu at (51.5, 68.6)
- added kibuzzard-672CB5CA: G***, kibuzzard-672CB5CA, B.Cu at (52.1, 71.1)
- added kibuzzard-672CB5D3: G***, kibuzzard-672CB5D3, B.Cu at (51.5, 73.7)
- added kibuzzard-672CB5DA: G***, kibuzzard-672CB5DA, B.Cu at (50.8, 76.2)
- added kibuzzard-672CB5E3: G***, kibuzzard-672CB5E3, B.Cu at (51.4, 78.7)
- added kibuzzard-672CB5EB: G***, kibuzzard-672CB5EB, B.Cu at (50.2, 81.3)
- added kibuzzard-672CB5F6: G***, kibuzzard-672CB5F6, B.Cu at (51.4, 83.8)
- added kibuzzard-672CB5FF: G***, kibuzzard-672CB5FF, B.Cu at (51.5, 86.4)
- added kibuzzard-672CB606: G***, kibuzzard-672CB606, B.Cu at (50.3, 88.9)
- added kibuzzard-672CB60E: G***, kibuzzard-672CB60E, B.Cu at (49.7, 91.4)
- added kibuzzard-672CB614: G***, kibuzzard-672CB614, B.Cu at (51.5, 94.0)
Other:
- board text added: "v1rev2"
- board text removed: "v1rev1"
