File: osc-board/osc-board.kicad_pcb (KiCad board)
At the start: 4 copper layers, 30.5 x 73.7 mm, 63 parts, among them J1 01x20, J2 01x20, J3 Conn_01x03_Female, J4 Conn_01x03_Female, Q1 MMBT3906, Q2 MMBT3906, U1 LM13700, U2 TL074, U3 TL074

Commit message: Carrier ordered
Parts:
- added G***: LOGO, LOGO, B.Cu at (99.1, 128.3)
- added REF**: OSHW-Logo2_7.3x6mm_SilkScreen, Symbol:OSHW-Logo2_7.3x6mm_SilkScreen, B.Cu at (99.1, 66.0)
- added kibuzzard-672CA102: G***, kibuzzard-672CA102, B.Cu at (106.8, 73.7)
- added kibuzzard-672CA109: G***, kibuzzard-672CA109, B.Cu at (106.8, 116.8)
- added kibuzzard-672CA109: G***, kibuzzard-672CA109, B.Cu at (106.8, 81.3)
- added kibuzzard-672CA109: G***, kibuzzard-672CA109, B.Cu at (106.8, 109.2)
- added kibuzzard-672CA109: G***, kibuzzard-672CA109, B.Cu at (106.8, 76.2)
- added kibuzzard-672CA109: G***, kibuzzard-672CA109, B.Cu at (106.8, 121.9)
- added kibuzzard-672CA109: G***, kibuzzard-672CA109, B.Cu at (106.8, 96.5)
- added kibuzzard-672CA109: G***, kibuzzard-672CA109, B.Cu at (106.8, 101.6)
- added kibuzzard-672CA109: G***, kibuzzard-672CA109, B.Cu at (106.8, 88.9)
- added kibuzzard-672CA10D: G***, kibuzzard-672CA10D, B.Cu at (106.8, 78.7)
- added kibuzzard-672CA24E: G***, kibuzzard-672CA24E, B.Cu at (91.3, 73.7)
- added kibuzzard-672CA252: G***, kibuzzard-672CA252, B.Cu at (91.2, 96.5)
- added kibuzzard-672CA252: G***, kibuzzard-672CA252, B.Cu at (91.2, 109.2)
- added kibuzzard-672CA252: G***, kibuzzard-672CA252, B.Cu at (91.3, 76.2)
- added kibuzzard-672CA252: G***, kibuzzard-672CA252, B.Cu at (91.2, 101.6)
- added kibuzzard-672CA252: G***, kibuzzard-672CA252, B.Cu at (91.2, 121.9)
- added kibuzzard-672CA252: G***, kibuzzard-672CA252, B.Cu at (91.2, 88.9)
- added kibuzzard-6771A5DA: G***, kibuzzard-6771A5DA, B.Cu at (105.5, 83.8)
- added kibuzzard-6771A5FD: G***, kibuzzard-6771A5FD, B.Cu at (92.5, 104.1)
- added kibuzzard-6771A890: G***, kibuzzard-6771A890, B.Cu at (105.7, 104.1)
- added kibuzzard-6771A943: G***, kibuzzard-6771A943, B.Cu at (106.8, 86.4)
- added kibuzzard-6771A949: G***, kibuzzard-6771A949, B.Cu at (91.2, 86.4)
- added kibuzzard-6771A969: G***, kibuzzard-6771A969, B.Cu at (106.9, 91.4)
- added kibuzzard-6771A96D: G***, kibuzzard-6771A96D, B.Cu at (91.7, 91.4)
- added kibuzzard-6771A9AC: G***, kibuzzard-6771A9AC, B.Cu at (106.9, 111.8)
- added kibuzzard-6771A9DB: G***, kibuzzard-6771A9DB, B.Cu at (91.2, 94.0)
- added kibuzzard-6771A9DE: G***, kibuzzard-6771A9DE, B.Cu at (107.4, 94.0)
- added kibuzzard-6771A9ED: G***, kibuzzard-6771A9ED, B.Cu at (107.4, 114.3)
- added kibuzzard-6771AA0E: G***, kibuzzard-6771AA0E, B.Cu at (91.7, 99.1)
- added kibuzzard-6771AA16: G***, kibuzzard-6771AA16, B.Cu at (106.9, 99.1)
- added kibuzzard-6771AA21: G***, kibuzzard-6771AA21, B.Cu at (106.9, 119.4)
- added kibuzzard-6771AA3E: G***, kibuzzard-6771AA3E, B.Cu at (91.2, 106.7)
- added kibuzzard-6771AA6F: G***, kibuzzard-6771AA6F, B.Cu at (106.8, 106.7)
- added kibuzzard-6776C4B6: G***, kibuzzard-6776C4B6, F.Cu at (99.1, 129.5)
Other:
- board text added: "1"
- board text added: "10"
- board text added: "11"
- board text added: "12"
- board text added: "13"
- board text added: "14"
- board text added: "15"
- board text added: "16"
- board text added: "17"
- board text added: "18"
- board text added: "19"
- board text added: "2"
- board text added: "20"
- board text added: "3"
- board text added: "4"
- board text added: "5"
- board text added: "6"
- board text added: "7"
- board text added: "8"
- board text added: "9"
- board text added: "pedalmarkt.com"
- board text added: "v1rev1"
